Commit message: Fixed bug where Controllers are not loading

File: install/hexapod_description/share/hexapod_description/robots/hexapod.urdf.xacro (robot description, xacro)
@@ -19,5 +19,5 @@
     <!-- Base -->
   <xacro:base parent="base_footprint">
-		<origin xyz="0 0 0" rpy="0 0 0"/>
+			<origin xyz="0 0 0.8" rpy="0 0 0"/>
   </xacro:base>
     <!-- Arm -->

File: install/hexapod_description/share/hexapod_description/ros2_control/hexapod.ros2_control.xacro (robot description, xacro)
@@ -2,4 +2,13 @@
 <robot
 	xmlns:xacro="http://www.ros.org/wiki/xacro">
+  <xacro:macro name="joint" params="name">
+    <joint name="${name}">
+				<command_interface name="position">
+					<param name="min">-1</param>
+					<param name="max">1</param>
+				</command_interface>
+				<state_interface name="position"/>
+			</joint>
+  </xacro:macro>
 	<xacro:macro name="hexapod_ros2_control">
 		<ros2_control name="GazeboSystem" type="system">
@@ -8,46 +17,25 @@
         <!-- <plugin>ros2_control_demo_example_1/RRBotSystemPositionOnlyHardware</plugin> -->
 			</hardware>
-			<joint name="arm_rotator_joint">
-				<command_interface name="position">
-					<param name="min">-1</param>
-					<param name="max">1</param>
-				</command_interface>
-				<state_interface name="position"/>
-			</joint>
-<joint name="arm_abductor_joint">
-				<command_interface name="position">
-					<param name="min">-1</param>
-					<param name="max">1</param>
-				</command_interface>
-				<state_interface name="position"/>
-			</joint>
-<joint name="arm_retractor_joint">
-				<command_interface name="position">
-					<param name="min">-1</param>
-					<param name="max">1</param>
-				</command_interface>
-				<state_interface name="position"/>
-			</joint>
-<joint name="top_left_rotate_joint">
-				<command_interface name="position">
-					<param name="min">-1</param>
-					<param name="max">1</param>
-				</command_interface>
-				<state_interface name="position"/>
-			</joint>
-<joint name="top_left_abduct_joint">
-				<command_interface name="position">
-					<param name="min">-1</param>
-					<param name="max">1</param>
-				</command_interface>
-				<state_interface name="position"/>
-			</joint>
-<joint name="top_left_retract_joint">
-				<command_interface name="position">
-					<param name="min">-1</param>
-					<param name="max">1</param>
-				</command_interface>
-				<state_interface name="position"/>
-			</joint>
+      <xacro:joint name="arm_rotator_joint"/>
+      <xacro:joint name="arm_abductor_joint"/>
+      <xacro:joint name="arm_retractor_joint"/>
+      <xacro:joint name="top_left_rotate_joint"/>
+      <xacro:joint name="top_left_abduct_joint"/>
+      <xacro:joint name="top_left_retract_joint"/>
+      <xacro:joint name="mid_left_rotate_joint"/>
+      <xacro:joint name="mid_left_abduct_joint"/>
+      <xacro:joint name="mid_left_retract_joint"/>
+      <xacro:joint name="bottom_left_rotate_joint"/>
+      <xacro:joint name="bottom_left_abduct_joint"/>
+      <xacro:joint name="bottom_left_retract_joint"/>
+      <xacro:joint name="top_right_rotate_joint"/>
+      <xacro:joint name="top_right_abduct_joint"/>
+      <xacro:joint name="top_right_retract_joint"/>
+      <xacro:joint name="mid_right_rotate_joint"/>
+      <xacro:joint name="mid_right_abduct_joint"/>
+      <xacro:joint name="mid_right_retract_joint"/>
+      <xacro:joint name="bottom_right_rotate_joint"/>
+      <xacro:joint name="bottom_right_abduct_joint"/>
+      <xacro:joint name="bottom_right_retract_joint"/>
 		</ros2_control>
 	</xacro:macro>
