Commit message: Changed world

File: install/hexapod_description/share/hexapod_description/gazebo/hexapod.gazebo.xacro (robot description, xacro)
@@ -3,12 +3,9 @@
   <xacro:macro name="hexapod_gazebo">
     <!-- =============== Gazebo =============== -->
-<gazebo>
-  <plugin filename="libgz_ros2_control-system" name="gz_ros2_control::GazeboSimROS2ControlPlugin">
-    <parameters>$(find hexapod_description)/config/hexapod_sim.yaml</parameters>
-  </plugin>
+    <gazebo>
       <plugin filename="gz-sim-sensors-system" name="gz::sim::systems::Sensors">
         <render_engine>ogre2</render_engine>
       </plugin>
-</gazebo>
+    </gazebo>
   </xacro:macro>
 </robot>

File: install/hexapod_description/share/hexapod_description/robots/hexapod.urdf.xacro (robot description, xacro)
@@ -5,47 +5,49 @@
   <xacro:property name="description_package" value="$(find hexapod_description)"/>
   <xacro:property name="robots" value="${description_package}/robots"/>
-  <xacro:property  name="meshes" value="file://$(find hexapod_description)/meshes"/>
-  <xacro:include filename="$(find hexapod_description)/gazebo/hexapod.gazebo.xacro" />
-  <xacro:include filename="$(find hexapod_description)/ros2_control/hexapod.ros2_control.xacro" />
-	<xacro:include filename="$(find hexapod_description)/materials/hexapod.materials.xacro" />
-	<xacro:include filename="$(find hexapod_description)/transmission/hexapod.trans.xacro" />
-  <xacro:include filename="${robots}/parts/base/base.urdf.xacro" />
-  <xacro:include filename="${robots}/parts/arm/arm.urdf.xacro" />
-  <xacro:include filename="${robots}/parts/leg/leg.urdf.xacro" />
-  <xacro:include filename="${robots}/parts/camera/camera.urdf.xacro" />
+  <xacro:property name="meshes" value="file://$(find hexapod_description)/meshes"/>
+  <xacro:include filename="$(find hexapod_description)/gazebo/hexapod.gazebo.xacro"/>
+  <xacro:include filename="$(find hexapod_description)/ros2_control/hexapod.ros2_control.xacro"/>
+  <xacro:include filename="$(find hexapod_description)/materials/hexapod.materials.xacro"/>
+  <xacro:include filename="${robots}/parts/base/base.urdf.xacro"/>
+  <xacro:include filename="${robots}/parts/arm/arm.urdf.xacro"/>
+  <xacro:include filename="${robots}/parts/leg/leg.urdf.xacro"/>
+  <xacro:include filename="${robots}/parts/camera/camera.urdf.xacro"/>
   <!-- =============== Link & Joint =============== -->
   <!-- Base -->
-  <link name="base_footprint"/> <!--link name="base_footprint"/ -->
-    <!-- Base -->
+  <link name="base_footprint"/>
+  <!--link name="base_footprint"/ -->
+  <!-- Base -->
   <xacro:base parent="base_footprint">
-			<origin xyz="0 0 0.8" rpy="0 0 0"/>
+    <origin xyz="0 0 0.8" rpy="0 0 0"/>
   </xacro:base>
-    <!-- Arm -->
-  <xacro:arm parent="base_link"> <origin xyz="0.025588 -0.019423 0.0449" rpy="0 0 0"/> </xacro:arm>
-    <!-- Camera -->
+  <!-- Arm -->
+  <xacro:arm parent="base_link">
+    <origin xyz="0.025588 -0.019423 0.0449" rpy="0 0 0"/>
+  </xacro:arm>
+  <!-- Camera -->
   <xacro:camera parent="arm_retractor">
-		<origin xyz="-0.081856 -0.02175 -0.054547" rpy="0 0 0"/>
+    <origin xyz="-0.081856 -0.02175 -0.054547" rpy="0 0 0"/>
   </xacro:camera>
-    <!-- Leg -->
+  <!-- Leg -->
   <xacro:leg parent="base_link" prefix="top_left">
     <origin xyz="0.074451 0.046824 0.0297" rpy="0 0 ${-1/4*M_PI}"/>
   </xacro:leg>
-    <!-- Leg -->
+  <!-- Leg -->
   <xacro:leg parent="base_link" prefix="mid_left">
     <origin xyz="0.003612 0.056729 0.0306" rpy="0 0 ${0}"/>
   </xacro:leg>
-    <!-- Leg -->
+  <!-- Leg -->
   <xacro:leg parent="base_link" prefix="bottom_left">
     <origin xyz="-0.067095 0.047401 0.0297" rpy="0 0 ${1/4*M_PI}"/>
   </xacro:leg>
-    <!-- Leg -->
+  <!-- Leg -->
   <xacro:leg parent="base_link" prefix="top_right">
-		<origin xyz="0.075633 -0.046741 0.0297" rpy="0 0 ${(1+1/4)*M_PI}"/>
+    <origin xyz="0.075633 -0.046741 0.0297" rpy="0 0 ${(1+1/4)*M_PI}"/>
   </xacro:leg>
-    <!-- Leg -->
+  <!-- Leg -->
   <xacro:leg parent="base_link" prefix="mid_right">
     <origin xyz="0.003574 -0.054899 0.0306" rpy="0 0 ${1*M_PI}"/>
   </xacro:leg>
-    <!-- Leg -->
+  <!-- Leg -->
   <xacro:leg parent="base_link" prefix="bottom_right">
     <origin xyz="-0.067095 -0.046741 0.0297" rpy="0 0 ${(1-1/4)*M_PI}"/>
@@ -54,3 +56,3 @@
   <xacro:hexapod_gazebo/>
   <xacro:hexapod_ros2_control/>
-  </robot>
+</robot>

File: install/hexapod_description/share/hexapod_description/robots/parts/arm/arm.urdf.xacro (robot description, xacro)
@@ -3,110 +3,110 @@
   <xacro:macro name="arm" params="parent *joint_origin">
     <!-- Joints -->
-		<joint name="arm_base_mount_joint" type="fixed">
-			<xacro:insert_block name="joint_origin"/>
-			<parent link="${parent}"/>
-		  <child link="arm_base"/>
-		</joint>
-	<joint name="arm_rotator_joint" type="continuous">
-		<origin xyz="8.8e-05 0.019999 0.02995" rpy="0 0 0"/>
-		<parent link="arm_base"/>
-		<child link="arm_rotator"/>
-		<axis xyz="0.0 -0.0 -1.0"/>
-	</joint>
-	<joint name="arm_abductor_joint" type="revolute">
-		<origin xyz="0.014582 0.00069 0.013923" rpy="0 0 0"/>
-		<parent link="arm_rotator"/>
-		<child link="arm_abductor"/>
-		<axis xyz="-1.0 0.0 -0.0"/>
-		<limit upper="1.570796" lower="-1.570796" effort="100" velocity="100"/>
-	</joint>
-	<joint name="arm_retractor_joint" type="revolute">
-		<origin xyz="-0.000401 0.0 0.046709" rpy="0 0 0"/>
-		<parent link="arm_abductor"/>
-		<child link="arm_retractor"/>
-		<axis xyz="-0.999993 0.0 -0.003676"/>
-		<limit upper="1.570796" lower="-1.570796" effort="100" velocity="100"/>
-	</joint>
-  <!-- Links -->
-	<link name="arm_rotator">
-		<inertial>
-			<origin xyz="-0.00046642883527773724 0.0027188082250819237 0.00576546998065737" rpy="0 0 0"/>
-			<mass value="0.02623546025799875"/>
-			<inertia ixx="4e-06" iyy="4e-06" izz="5e-06" ixy="0.0" iyz="-0.0" ixz="0.0"/>
-		</inertial>
-		<visual>
-			<origin xyz="-0.025676 -0.000576 -0.07485" rpy="0 0 0"/>
-			<geometry>
+    <joint name="arm_base_mount_joint" type="fixed">
+      <xacro:insert_block name="joint_origin"/>
+      <parent link="${parent}"/>
+      <child link="arm_base"/>
+    </joint>
+    <joint name="arm_rotator_joint" type="continuous">
+      <origin xyz="8.8e-05 0.019999 0.02995" rpy="0 0 0"/>
+      <parent link="arm_base"/>
+      <child link="arm_rotator"/>
+      <axis xyz="0.0 -0.0 -1.0"/>
+    </joint>
+    <joint name="arm_abductor_joint" type="revolute">
+      <origin xyz="0.014582 0.00069 0.013923" rpy="0 0 0"/>
+      <parent link="arm_rotator"/>
+      <child link="arm_abductor"/>
+      <axis xyz="-1.0 0.0 -0.0"/>
+      <limit upper="1.570796" lower="-1.570796" effort="100" velocity="100"/>
+    </joint>
+    <joint name="arm_retractor_joint" type="revolute">
+      <origin xyz="-0.000401 0.0 0.046709" rpy="0 0 0"/>
+      <parent link="arm_abductor"/>
+      <child link="arm_retractor"/>
+      <axis xyz="-0.999993 0.0 -0.003676"/>
+      <limit upper="1.570796" lower="-1.570796" effort="100" velocity="100"/>
+    </joint>
+    <!-- Links -->
+    <link name="arm_rotator">
+      <inertial>
+        <origin xyz="-0.00046642883527773724 0.0027188082250819237 0.00576546998065737" rpy="0 0 0"/>
+        <mass value="0.02623546025799875"/>
+        <inertia ixx="4e-06" iyy="4e-06" izz="5e-06" ixy="0.0" iyz="-0.0" ixz="0.0"/>
+      </inertial>
+      <visual>
+        <origin xyz="-0.025676 -0.000576 -0.07485" rpy="0 0 0"/>
+        <geometry>
           <mesh filename="${meshes}/arm/rotator.stl" scale="0.001 0.001 0.001"/>
-			</geometry>
-			<material name="dark"/>
-		</visual>
-		<collision>
-			<origin xyz="-0.025676 -0.000576 -0.07485" rpy="0 0 0"/>
-			<geometry>
+        </geometry>
+        <material name="dark"/>
+      </visual>
+      <collision>
+        <origin xyz="-0.025676 -0.000576 -0.07485" rpy="0 0 0"/>
+        <geometry>
           <mesh filename="${meshes}/arm/rotator.stl" scale="0.001 0.001 0.001"/>
-			</geometry>
-		</collision>
-	</link>
-	<link name="arm_abductor">
-		<inertial>
-			<origin xyz="-0.014167725035919117 3.5639852713031765e-07 0.031090662760010462" rpy="0 0 0"/>
-			<mass value="0.016534189067873267"/>
-			<inertia ixx="5e-06" iyy="7e-06" izz="2e-06" ixy="-0.0" iyz="-0.0" ixz="1e-06"/>
-		</inertial>
-		<visual>
-			<origin xyz="-0.040258 -0.001266 -0.088773" rpy="0 0 0"/>
-			<geometry>
+        </geometry>
+      </collision>
+    </link>
+    <link name="arm_abductor">
+      <inertial>
+        <origin xyz="-0.014167725035919117 3.5639852713031765e-07 0.031090662760010462" rpy="0 0 0"/>
+        <mass value="0.016534189067873267"/>
+        <inertia ixx="5e-06" iyy="7e-06" izz="2e-06" ixy="-0.0" iyz="-0.0" ixz="1e-06"/>
+      </inertial>
+      <visual>
+        <origin xyz="-0.040258 -0.001266 -0.088773" rpy="0 0 0"/>
+        <geometry>
           <mesh filename="${meshes}/arm/abductor.stl" scale="0.001 0.001 0.001"/>
-			</geometry>
-			<material name="dark"/>
-		</visual>
-		<collision>
-			<origin xyz="-0.040258 -0.001266 -0.088773" rpy="0 0 0"/>
-			<geometry>
+        </geometry>
+        <material name="dark"/>
+      </visual>
+      <collision>
+        <origin xyz="-0.040258 -0.001266 -0.088773" rpy="0 0 0"/>
+        <geometry>
           <mesh filename="${meshes}/arm/abductor.stl" scale="0.001 0.001 0.001"/>
-			</geometry>
-		</collision>
-	</link>
-	<link name="arm_retractor">
-		<inertial>
-			<origin xyz="-0.011027322351092845 -5.220911472792085e-05 0.023364114206742087" rpy="0 0 0"/>
-			<mass value="0.015328010788351278"/>
-			<inertia ixx="3e-06" iyy="5e-06" izz="4e-06" ixy="0.0" iyz="0.0" ixz="-0.0"/>
-		</inertial>
-		<visual>
-			<origin xyz="-0.039857 -0.001266 -0.135482" rpy="0 0 0"/>
-			<geometry>
+        </geometry>
+      </collision>
+    </link>
+    <link name="arm_retractor">
+      <inertial>
+        <origin xyz="-0.011027322351092845 -5.220911472792085e-05 0.023364114206742087" rpy="0 0 0"/>
+        <mass value="0.015328010788351278"/>
+        <inertia ixx="3e-06" iyy="5e-06" izz="4e-06" ixy="0.0" iyz="0.0" ixz="-0.0"/>
+      </inertial>
+      <visual>
+        <origin xyz="-0.039857 -0.001266 -0.135482" rpy="0 0 0"/>
+        <geometry>
           <mesh filename="${meshes}/arm/retractor.stl" scale="0.001 0.001 0.001"/>
-			</geometry>
-			<material name="dark"/>
-		</visual>
-		<collision>
-			<origin xyz="-0.039857 -0.001266 -0.135482" rpy="0 0 0"/>
-			<geometry>
+        </geometry>
+        <material name="dark"/>
+      </visual>
+      <collision>
+        <origin xyz="-0.039857 -0.001266 -0.135482" rpy="0 0 0"/>
+        <geometry>
           <mesh filename="${meshes}/arm/retractor.stl" scale="0.001 0.001 0.001"/>
-			</geometry>
-		</collision>
-	</link>
-	<link name="arm_base">
-		<inertial>
-			<origin xyz="0.004115093716825637 0.020000308654227843 0.01035421864114821" rpy="0 0 0"/>
-			<mass value="0.014628769254330782"/>
-			<inertia ixx="2e-06" iyy="3e-06" izz="2e-06" ixy="0.0" iyz="0.0" ixz="-0.0"/>
-		</inertial>
-		<visual>
-			<origin xyz="-0.025588 0.019423 -0.0449" rpy="0 0 0"/>
-			<geometry>
+        </geometry>
+      </collision>
+    </link>
+    <link name="arm_base">
+      <inertial>
+        <origin xyz="0.004115093716825637 0.020000308654227843 0.01035421864114821" rpy="0 0 0"/>
+        <mass value="0.014628769254330782"/>
+        <inertia ixx="2e-06" iyy="3e-06" izz="2e-06" ixy="0.0" iyz="0.0" ixz="-0.0"/>
+      </inertial>
+      <visual>
+        <origin xyz="-0.025588 0.019423 -0.0449" rpy="0 0 0"/>
+        <geometry>
           <mesh filename="${meshes}/arm/base.stl" scale="0.001 0.001 0.001"/>
-			</geometry>
-			<material name="dark"/>
-		</visual>
-		<collision>
-			<origin xyz="-0.025588 0.019423 -0.0449" rpy="0 0 0"/>
-			<geometry>
+        </geometry>
+        <material name="dark"/>
+      </visual>
+      <collision>
+        <origin xyz="-0.025588 0.019423 -0.0449" rpy="0 0 0"/>
+        <geometry>
           <mesh filename="${meshes}/arm/base.stl" scale="0.001 0.001 0.001"/>
-			</geometry>
-		</collision>
-	</link>
+        </geometry>
+      </collision>
+    </link>
   </xacro:macro>
 </robot>

File: install/hexapod_description/share/hexapod_description/robots/parts/base/base.urdf.xacro (robot description, xacro)
@@ -1,39 +1,38 @@
 <?xml version="1.0"?>
-<robot
-	xmlns:xacro="http://ros.org/wiki/xacro">
-	<xacro:macro name="base" params="parent *joint_origin">
+<robot xmlns:xacro="http://ros.org/wiki/xacro">
+  <xacro:macro name="base" params="parent *joint_origin">
     <!-- Joints -->
-		<joint name="base_link_joint" type="fixed">
-			<xacro:insert_block name="joint_origin"/>
-			<parent link="${parent}"/>
-			<child link="base_link"/>
-		</joint>
-      <!-- Links -->
-		<link name="base_link">
-			<inertial>
-				<origin xyz="0.005334608688478278 0.0002689766590861973 0.0184918721125776" rpy="0 0 0"/>
-				<mass value="0.1730647056842735"/>
-				<inertia ixx="0.000266" iyy="0.000406" izz="0.0006" ixy="4e-06" iyz="-0.0" ixz="-1e-06"/>
-			</inertial>
-			<visual>
-				<origin xyz="0 0 0" rpy="0 0 0"/>
-				<geometry>
+    <joint name="base_link_joint" type="fixed">
+      <xacro:insert_block name="joint_origin"/>
+      <parent link="${parent}"/>
+      <child link="base_link"/>
+    </joint>
+    <!-- Links -->
+    <link name="base_link">
+      <inertial>
+        <origin xyz="0.005334608688478278 0.0002689766590861973 0.0184918721125776" rpy="0 0 0"/>
+        <mass value="0.1730647056842735"/>
+        <inertia ixx="0.000266" iyy="0.000406" izz="0.0006" ixy="4e-06" iyz="-0.0" ixz="-1e-06"/>
+      </inertial>
+      <visual>
+        <origin xyz="0 0 0" rpy="0 0 0"/>
+        <geometry>
           <mesh filename="${meshes}/base/base_link.stl" scale="0.001 0.001 0.001"/>
-				</geometry>
-				<material name="dark"/>
-			</visual>
-			<collision>
-				<origin xyz="0 0 0" rpy="0 0 0"/>
-				<geometry>
+        </geometry>
+        <material name="dark"/>
+      </visual>
+      <collision>
+        <origin xyz="0 0 0" rpy="0 0 0"/>
+        <geometry>
           <mesh filename="${meshes}/base/base_link.stl" scale="0.001 0.001 0.001"/>
-				</geometry>
-			</collision>
-		</link>
-      <!-- Gazebo Properties -->
-		<gazebo reference="base_link">
-			<selfCollide>false</selfCollide>
-			<mu1 value="0.05" />
-			<mu2 value="0.05" />
-		</gazebo>
-	</xacro:macro>
+        </geometry>
+      </collision>
+    </link>
+    <!-- Gazebo Properties -->
+    <gazebo reference="base_link">
+      <selfCollide>false</selfCollide>
+      <mu1 value="0.05"/>
+      <mu2 value="0.05"/>
+    </gazebo>
+  </xacro:macro>
 </robot>

File: install/hexapod_description/share/hexapod_description/robots/parts/camera/camera.urdf.xacro (robot description, xacro)
@@ -1,65 +1,64 @@
-<?xml version="1.0" ?>
-<robot name="hexapod_waffle"
-	xmlns:xacro="http://ros.org/wiki/xacro">
-	<xacro:property name="r200_cam_rgb_px" value="0.005"/>
-	<xacro:property name="r200_cam_rgb_py" value="0.018"/>
-	<xacro:property name="r200_cam_rgb_pz" value="0.013"/>
-	<xacro:property name="r200_cam_depth_offset" value="0.01"/>
-	<xacro:macro name="camera" params="parent *joint_origin">
+<?xml version="1.0"?>
+<robot xmlns:xacro="http://ros.org/wiki/xacro" name="hexapod_waffle">
+  <xacro:property name="r200_cam_rgb_px" value="0.005"/>
+  <xacro:property name="r200_cam_rgb_py" value="0.018"/>
+  <xacro:property name="r200_cam_rgb_pz" value="0.013"/>
+  <xacro:property name="r200_cam_depth_offset" value="0.01"/>
+  <xacro:macro name="camera" params="parent *joint_origin">
     <!-- Joints -->
-		<joint name="camera_case_mount" type="fixed">
-			<xacro:insert_block name="joint_origin"/>
-			<parent link="${parent}"/>
-			<child link="camera_link"/>
-		</joint>
-      <!-- Links -->
-	<link name="camera_link">
-		<inertial>
-			<origin xyz="0.07257325961305607 0.023187735063927437 0.09454807900867684" rpy="0 0 0"/>
-			<mass value="0.00672643608404174"/>
-			<inertia ixx="1e-06" iyy="2e-06" izz="3e-06" ixy="0.0" iyz="0.0" ixz="0.0"/>
-		</inertial>
-		<visual>
-			<origin xyz="0.041999 0.020484 -0.080935" rpy="0 0 0"/>
-			<geometry>
+    <joint name="camera_case_mount" type="fixed">
+      <xacro:insert_block name="joint_origin"/>
+      <parent link="${parent}"/>
+      <child link="camera_link"/>
+    </joint>
+    <!-- Links -->
+    <link name="camera_link">
+      <inertial>
+        <origin xyz="0.07257325961305607 0.023187735063927437 0.09454807900867684" rpy="0 0 0"/>
+        <mass value="0.00672643608404174"/>
+        <inertia ixx="1e-06" iyy="2e-06" izz="3e-06" ixy="0.0" iyz="0.0" ixz="0.0"/>
+      </inertial>
+      <visual>
+        <origin xyz="0.041999 0.020484 -0.080935" rpy="0 0 0"/>
+        <geometry>
           <mesh filename="${meshes}/sensors/camera/camera.stl" scale="0.001 0.001 0.001"/>
-			</geometry>
-			<material name="red"/>
-		</visual>
-		<collision>
-			<origin xyz="0.041999 0.020484 -0.080935" rpy="0 0 0"/>
-			<geometry>
+        </geometry>
+        <material name="red"/>
+      </visual>
+      <collision>
+        <origin xyz="0.041999 0.020484 -0.080935" rpy="0 0 0"/>
+        <geometry>
           <mesh filename="${meshes}/sensors/camera/camera.stl" scale="0.001 0.001 0.001"/>
-			</geometry>
-		</collision>
-  </link>
-      <!-- Gazebo -->
-  <gazebo reference="camera_link">
-    <sensor name="depth_camera" type="depth_camera">
-      <always_on>true</always_on>
-      <visualize>true</visualize>
-      <update_rate>60</update_rate>
-      <topic>depth_camera/depth/image_raw</topic>
-      <frame_id>camera_depth_frame</frame_id>
-      <camera name="sipeed Max A10">
-        <camera_info_topic>depth_camera/depth/camera_info</camera_info_topic>
-        <horizontal_fov>1.02974</horizontal_fov>
-        <image>
-          <width>1920</width>
-          <height>1080</height>
+        </geometry>
+      </collision>
+    </link>
+    <!-- Gazebo -->
+    <gazebo reference="camera_link">
+      <sensor name="depth_camera" type="depth_camera">
+        <always_on>true</always_on>
+        <visualize>true</visualize>
+        <update_rate>60</update_rate>
+        <topic>depth_camera/depth/image_raw</topic>
+        <frame_id>camera_depth_frame</frame_id>
+        <camera name="sipeed Max A10">
+          <camera_info_topic>depth_camera/depth/camera_info</camera_info_topic>
+          <horizontal_fov>1.02974</horizontal_fov>
+          <image>
+            <width>1920</width>
+            <height>1080</height>
             <format>R_FLOAT32</format>
-        </image>
-        <clip>
-          <near>0.02</near>
-          <far>300</far>
-        </clip>
-        <noise>
-          <type>gaussian</type>
-          <mean>0.0</mean>
-          <stddev>0.007</stddev>
-        </noise>
-      </camera>
-    </sensor>
-  </gazebo>
-</xacro:macro>
+          </image>
+          <clip>
+            <near>0.02</near>
+            <far>300</far>
+          </clip>
+          <noise>
+            <type>gaussian</type>
+            <mean>0.0</mean>
+            <stddev>0.007</stddev>
+          </noise>
+        </camera>
+      </sensor>
+    </gazebo>
+  </xacro:macro>
 </robot>
