Commit message: Changed world

File: install/hexapod_description/share/hexapod_description/robots/parts/leg/leg.urdf.xacro (robot description, xacro)
@@ -4,114 +4,114 @@
     <!-- Joints -->
     <joint name="${prefix}_rotate_joint" type="revolute">
-			<xacro:insert_block name="joint_origin"/>
-			<parent link="${parent}"/>
+      <xacro:insert_block name="joint_origin"/>
+      <parent link="${parent}"/>
       <child link="${prefix}_cox"/>
-		  <axis xyz="-0.0 0.0 -1.0"/>
-		<limit upper="1.570796" lower="-1.570796" effort="100" velocity="100"/>
-		</joint>
+      <axis xyz="-0.0 0.0 -1.0"/>
+      <limit upper="1.570796" lower="-1.570796" effort="100" velocity="100"/>
+    </joint>
     <joint name="${prefix}_abduct_joint" type="revolute">
-		<origin xyz="0.020937 0.03 -0.021804" rpy="0 0 0"/>
-		<axis xyz="-1.0 -0.0 -0.0"/>
-		<limit upper="1.570796" lower="-1.570796" effort="100" velocity="100"/>
-		<parent link="${prefix}_cox"/>
-		<child link="${prefix}_femur"/>
-	</joint>
+      <origin xyz="0.020937 0.03 -0.021804" rpy="0 0 0"/>
+      <axis xyz="-1.0 -0.0 -0.0"/>
+      <limit upper="1.570796" lower="-1.570796" effort="100" velocity="100"/>
+      <parent link="${prefix}_cox"/>
+      <child link="${prefix}_femur"/>
+    </joint>
     <joint name="${prefix}_retract_joint" type="revolute">
-		<origin xyz="-0.029923 0.039696 -0.018563" rpy="0 0 0"/>
-		<parent link="${prefix}_femur"/>
-		<child link="${prefix}_tibia"/>
-		<axis xyz="0.707029 0.707185 0.0"/>
-		<limit upper="1.570796" lower="-1.570796" effort="100" velocity="100"/>
-	</joint>
+      <origin xyz="-0.029923 0.039696 -0.018563" rpy="0 0 0"/>
+      <parent link="${prefix}_femur"/>
+      <child link="${prefix}_tibia"/>
+      <axis xyz="0.707029 0.707185 0.0"/>
+      <limit upper="1.570796" lower="-1.570796" effort="100" velocity="100"/>
+    </joint>
     <link name="${prefix}_cox">
-		<inertial>
-			<origin xyz="0.0012733261090569089 0.014903434394979126 -0.02034582182041162" rpy="0 0 0"/>
-			<mass value="0.01391683496290758"/>
-			<inertia ixx="3e-06" iyy="4e-06" izz="3e-06" ixy="-0.0" iyz="0.0" ixz="0.0"/>
-		</inertial>
-		<visual>
-			<origin xyz="-0.003612 -0.056729 -0.0306" rpy="0 0 0"/>
-			<geometry>
+      <inertial>
+        <origin xyz="0.0012733261090569089 0.014903434394979126 -0.02034582182041162" rpy="0 0 0"/>
+        <mass value="0.01391683496290758"/>
+        <inertia ixx="3e-06" iyy="4e-06" izz="3e-06" ixy="-0.0" iyz="0.0" ixz="0.0"/>
+      </inertial>
+      <visual>
+        <origin xyz="-0.003612 -0.056729 -0.0306" rpy="0 0 0"/>
+        <geometry>
           <mesh filename="${meshes}/leg/cox_left_mid.stl" scale="0.001 0.001 0.001"/>
-			</geometry>
-			<material name="dark"/>
-		</visual>
-		<collision>
-			<origin xyz="-0.003612 -0.056729 -0.0306" rpy="0 0 0"/>
-			<geometry>
+        </geometry>
+        <material name="dark"/>
+      </visual>
+      <collision>
+        <origin xyz="-0.003612 -0.056729 -0.0306" rpy="0 0 0"/>
+        <geometry>
           <mesh filename="${meshes}/leg/cox_left_mid.stl" scale="0.001 0.001 0.001"/>
-			</geometry>
-		</collision>
-	</link>
+        </geometry>
+      </collision>
+    </link>
     <link name="${prefix}_tibia">
-		<inertial>
-			<origin xyz="0.015589179677926173 0.010695585608516162 -0.0223992522730315" rpy="0 0 0"/>
-			<mass value="0.012279438354877548"/>
-			<inertia ixx="5e-06" iyy="6e-06" izz="2e-06" ixy="0.0" iyz="-1e-06" ixz="0.0"/>
-		</inertial>
-		<visual>
-			<origin xyz="0.005374 -0.126425 0.009767" rpy="0 0 0"/>
-			<geometry>
+      <inertial>
+        <origin xyz="0.015589179677926173 0.010695585608516162 -0.0223992522730315" rpy="0 0 0"/>
+        <mass value="0.012279438354877548"/>
+        <inertia ixx="5e-06" iyy="6e-06" izz="2e-06" ixy="0.0" iyz="-1e-06" ixz="0.0"/>
+      </inertial>
+      <visual>
+        <origin xyz="0.005374 -0.126425 0.009767" rpy="0 0 0"/>
+        <geometry>
           <mesh filename="${meshes}/leg/tibia_left_mid.stl" scale="0.001 0.001 0.001"/>
-			</geometry>
-			<material name="dark"/>
-		</visual>
-		<collision>
-			<origin xyz="0.005374 -0.126425 0.009767" rpy="0 0 0"/>
-			<geometry>
+        </geometry>
+        <material name="dark"/>
+      </visual>
+      <collision>
+        <origin xyz="0.005374 -0.126425 0.009767" rpy="0 0 0"/>
+        <geometry>
           <mesh filename="${meshes}/leg/tibia_left_mid.stl" scale="0.001 0.001 0.001"/>
-			</geometry>
-		</collision>
-	</link>
+        </geometry>
+      </collision>
+    </link>
     <link name="${prefix}_femur">
-		<inertial>
-			<origin xyz="-0.015011654934717145 0.020989624323966824 -0.005728252734904802" rpy="0 0 0"/>
-			<mass value="0.018823784549799234"/>
-			<inertia ixx="5e-06" iyy="3e-06" izz="5e-06" ixy="0.0" iyz="2e-06" ixz="-0.0"/>
-		</inertial>
-		<visual>
-			<origin xyz="-0.024549 -0.086729 -0.008796" rpy="0 0 0"/>
-			<geometry>
+      <inertial>
+        <origin xyz="-0.015011654934717145 0.020989624323966824 -0.005728252734904802" rpy="0 0 0"/>
+        <mass value="0.018823784549799234"/>
+        <inertia ixx="5e-06" iyy="3e-06" izz="5e-06" ixy="0.0" iyz="2e-06" ixz="-0.0"/>
+      </inertial>
+      <visual>
+        <origin xyz="-0.024549 -0.086729 -0.008796" rpy="0 0 0"/>
+        <geometry>
           <mesh filename="${meshes}/leg/femur_left_mid.stl" scale="0.001 0.001 0.001"/>
-			</geometry>
-			<material name="dark"/>
-		</visual>
-		<collision>
-			<origin xyz="-0.024549 -0.086729 -0.008796" rpy="0 0 0"/>
-			<geometry>
+        </geometry>
+        <material name="dark"/>
+      </visual>
+      <collision>
+        <origin xyz="-0.024549 -0.086729 -0.008796" rpy="0 0 0"/>
+        <geometry>
           <mesh filename="${meshes}/leg/femur_left_mid.stl" scale="0.001 0.001 0.001"/>
-			</geometry>
-		</collision>
-	</link>
-<transmission name="${prefix}_rotate_joint_tran">
-  <type>transmission_interface/SimpleTransmission</type>
-  <joint name="${prefix}_rotate_joint">
-    <hardwareInterface>hardware_interface/EffortJointInterface</hardwareInterface>
-  </joint>
-  <actuator name="${prefix}_rotate_joint_actr">
-    <hardwareInterface>hardware_interface/EffortJointInterface</hardwareInterface>
-    <mechanicalReduction>1</mechanicalReduction>
-  </actuator>
-</transmission>
-<transmission name="${prefix}_abduct_joint_tran">
-  <type>transmission_interface/SimpleTransmission</type>
-  <joint name="${prefix}_abduct_joint">
-    <hardwareInterface>hardware_interface/EffortJointInterface</hardwareInterface>
-  </joint>
-  <actuator name="${prefix}_abduct_joint_actr">
-    <hardwareInterface>hardware_interface/EffortJointInterface</hardwareInterface>
-    <mechanicalReduction>1</mechanicalReduction>
-  </actuator>
-</transmission>
-<transmission name="${prefix}_retract_joint_tran">
-  <type>transmission_interface/SimpleTransmission</type>
-  <joint name="${prefix}_retract_joint">
-    <hardwareInterface>hardware_interface/EffortJointInterface</hardwareInterface>
-  </joint>
-  <actuator name="${prefix}_retract_joint_actr">
-    <hardwareInterface>hardware_interface/EffortJointInterface</hardwareInterface>
-    <mechanicalReduction>1</mechanicalReduction>
-  </actuator>
-</transmission>
+        </geometry>
+      </collision>
+    </link>
+    <transmission name="${prefix}_rotate_joint_tran">
+      <type>transmission_interface/SimpleTransmission</type>
+      <joint name="${prefix}_rotate_joint">
+        <hardwareInterface>hardware_interface/EffortJointInterface</hardwareInterface>
+      </joint>
+      <actuator name="${prefix}_rotate_joint_actr">
+        <hardwareInterface>hardware_interface/EffortJointInterface</hardwareInterface>
+        <mechanicalReduction>1</mechanicalReduction>
+      </actuator>
+    </transmission>
+    <transmission name="${prefix}_abduct_joint_tran">
+      <type>transmission_interface/SimpleTransmission</type>
+      <joint name="${prefix}_abduct_joint">
+        <hardwareInterface>hardware_interface/EffortJointInterface</hardwareInterface>
+      </joint>
+      <actuator name="${prefix}_abduct_joint_actr">
+        <hardwareInterface>hardware_interface/EffortJointInterface</hardwareInterface>
+        <mechanicalReduction>1</mechanicalReduction>
+      </actuator>
+    </transmission>
+    <transmission name="${prefix}_retract_joint_tran">
+      <type>transmission_interface/SimpleTransmission</type>
+      <joint name="${prefix}_retract_joint">
+        <hardwareInterface>hardware_interface/EffortJointInterface</hardwareInterface>
+      </joint>
+      <actuator name="${prefix}_retract_joint_actr">
+        <hardwareInterface>hardware_interface/EffortJointInterface</hardwareInterface>
+        <mechanicalReduction>1</mechanicalReduction>
+      </actuator>
+    </transmission>
   </xacro:macro>
 </robot>

File: install/hexapod_description/share/hexapod_description/ros2_control/hexapod.ros2_control.xacro (robot description, xacro)
@@ -1,20 +1,23 @@
 <?xml version="1.0"?>
-<robot
-	xmlns:xacro="http://www.ros.org/wiki/xacro">
+<robot xmlns:xacro="http://www.ros.org/wiki/xacro">
   <xacro:macro name="joint" params="name">
     <joint name="${name}">
-				<command_interface name="position">
-					<param name="min">-1</param>
-					<param name="max">1</param>
-				</command_interface>
-				<state_interface name="position"/>
-			</joint>
+      <command_interface name="position">
+        <param name="min">-1</param>
+        <param name="max">1</param>
+      </command_interface>
+      <state_interface name="position"/>
+    </joint>
   </xacro:macro>
-	<xacro:macro name="hexapod_ros2_control">
-		<ros2_control name="GazeboSystem" type="system">
-			<hardware>
-				<plugin>gz_ros2_control/GazeboSimSystem</plugin>
-        <!-- <plugin>ros2_control_demo_example_1/RRBotSystemPositionOnlyHardware</plugin> -->
-			</hardware>
+  <gazebo>
+    <plugin filename="libgz_ros2_control-system" name="gz_ros2_control::GazeboSimROS2ControlPlugin">
+      <parameters>$(find hexapod_description)/config/hexapod_controllers.yaml</parameters>
+    </plugin>
+  </gazebo>
+  <xacro:macro name="hexapod_ros2_control">
+    <ros2_control name="GazeboSystem" type="system">
+      <hardware>
+        <plugin>gz_ros2_control/GazeboSimSystem</plugin>
+      </hardware>
       <xacro:joint name="arm_rotator_joint"/>
       <xacro:joint name="arm_abductor_joint"/>
@@ -38,5 +41,5 @@
       <xacro:joint name="bottom_right_abduct_joint"/>
       <xacro:joint name="bottom_right_retract_joint"/>
-		</ros2_control>
-	</xacro:macro>
+    </ros2_control>
+  </xacro:macro>
 </robot>
