Commit message: Connected between joint states and rviz2

File: src/hexapod_description/robots/parts/arm/arm.urdf.xacro (robot description, xacro)
@@ -13,4 +13,5 @@
       <child link="arm_rotator"/>
       <axis xyz="0.0 -0.0 -1.0"/>
+      <limit upper="1.570796" lower="-1.570796" effort="100" velocity="100"/>
     </joint>
     <joint name="arm_abductor_joint" type="revolute">
