Commit message: Transposed table

File: src/hexapod_description/robots/parts/camera/camera.urdf.xacro (robot description, xacro)
@@ -24,5 +24,5 @@
           <mesh filename="${meshes}/sensors/camera/camera.stl" scale="0.001 0.001 0.001"/>
         </geometry>
-        <material name="red"/>
+        <material name="dark"/>
       </visual>
       <collision>
@@ -41,5 +41,5 @@
         <topic>depth_camera/depth/image_raw</topic>
         <frame_id>camera_depth_frame</frame_id>
-        <camera name="sipeed Max A10">
+        <camera name="Sipeed MaixSense A10">
           <camera_info_topic>depth_camera/depth/camera_info</camera_info_topic>
           <horizontal_fov>1.02974</horizontal_fov>

Commit message: Fixed camera frame perspective

File: src/hexapod_description/robots/parts/camera/camera.urdf.xacro (robot description, xacro)
@@ -7,5 +7,5 @@
   <xacro:macro name="camera" params="parent *joint_origin">
     <!-- Joints -->
-    <joint name="camera_case_mount" type="fixed">
+    <joint name="camera_case_cover_joint" type="fixed">
       <xacro:insert_block name="joint_origin"/>
       <parent link="${parent}"/>
@@ -13,5 +13,5 @@
     </joint>
     <!-- Joints -->
-    <joint name="camera_mount" type="fixed">
+    <joint name="depth_camera_link_joint" type="fixed">
       <xacro:insert_block name="joint_origin"/>
       <parent link="${parent}"/>
@@ -48,4 +48,12 @@
     </visual>
     </link>
+    <!-- Joints -->
+    <joint name="depth_camera_optical_joint" type="fixed">
+      <origin xyz="0.0 0.0 0.0" rpy="${-pi/2} 0 ${-pi/2}"/>
+      <parent link="depth_camera_link"/>
+      <child link="depth_camera_optical_frame"/>
+    </joint>
+    <link name="depth_camera_optical_frame">
+    </link>
     <!-- Gazebo -->
 <gazebo reference="depth_camera_link">
@@ -55,5 +63,5 @@
     <update_rate>10</update_rate> <!-- Max FPS according to spec -->
     <topic>depth_camera/depth/image_raw</topic>
-    <gz_frame_id>depth_camera_link</gz_frame_id>
+    <gz_frame_id>depth_camera_optical_frame</gz_frame_id>
     <camera name="Sipeed_MaixSense_A010">
       <camera_info_topic>depth_camera/depth/camera_info</camera_info_topic>
