Commit message: Added Point markers relative to feet, added feet

File: src/hexapod_description/robots/parts/leg/leg.urdf.xacro (robot description, xacro)
@@ -23,4 +23,9 @@
       <axis xyz="1.0 0.00011 0.0"/>
       <limit upper="1.570796" lower="-1.570796" effort="100" velocity="100"/>
+    </joint>
+    <joint name="${prefix}_foot_joint" type="fixed">
+      <origin xyz="0.016 0.0 -0.07" rpy="0 0 0"/>
+      <parent link="${prefix}_tibia"/>
+      <child link="${prefix}_foot"/>
     </joint>
     <link name="${prefix}_cox">
@@ -63,4 +68,13 @@
         </geometry>
       </collision>
+    </link>
+    <link name="${prefix}_foot">
+      <visual>
+        <origin xyz="0.0 0.0 0.0" rpy="0 0 0"/>
+        <geometry>
+          <sphere  radius="0.0080"/>
+        </geometry>
+        <material name="dark"/>
+      </visual>
     </link>
     <link name="${prefix}_femur">
