Commit message: Fixed URDF, reorganized folder, added feet, added point markers

File: src/hexapod_description/materials/hexapod.materials.xacro (robot description, xacro)
@@ -3,33 +3,9 @@
   xmlns:xacro="http://ros.org/wiki/xacro">
   <!-- Init colour -->
-  <material name="black">
+  <material name="TPU">
     <color rgba="0.0 0.0 0.0 1.0"/>
   </material>
-  <material name="dark">
+  <material name="PLA">
     <color rgba="0.3 0.3 0.3 1.0"/>
   </material>
-  <material name="light_black">
-    <color rgba="0.4 0.4 0.4 1.0"/>
-  </material>
-  <material name="blue">
-    <color rgba="0.0 0.0 0.8 1.0"/>
-  </material>
-  <material name="green">
-    <color rgba="0.0 0.8 0.0 1.0"/>
-  </material>
-  <material name="grey">
-    <color rgba="0.5 0.5 0.5 1.0"/>
-  </material>
-  <material name="orange">
-    <color rgba="${255/255} ${108/255} ${10/255} 1.0"/>
-  </material>
-  <material name="brown">
-    <color rgba="${222/255} ${207/255} ${195/255} 1.0"/>
-  </material>
-  <material name="red">
-    <color rgba="0.8 0.0 0.0 1.0"/>
-  </material>
-  <material name="white">
-    <color rgba="1.0 1.0 1.0 1.0"/>
-  </material>
 </robot>

File: src/hexapod_description/robots/hexapod.urdf.xacro (robot description, xacro)
@@ -28,25 +28,25 @@
   </xacro:arm>
   <!-- Leg -->
-  <xacro:leg parent="base_link" prefix="top_left">
+  <xacro:leg parent="base_link" position="top" side="left">
     <origin xyz="0.074451 0.046824 0.0297" rpy="0 0 ${-1/4*pi}"/>
   </xacro:leg>
   <!-- Leg -->
-  <xacro:leg parent="base_link" prefix="mid_left">
+  <xacro:leg parent="base_link" position="mid" side="left">
     <origin xyz="0.003612 0.056729 0.0306" rpy="0 0 ${0}"/>
   </xacro:leg>
   <!-- Leg -->
-  <xacro:leg parent="base_link" prefix="bottom_left">
+  <xacro:leg parent="base_link" position="bottom" side="left">
     <origin xyz="-0.067095 0.047401 0.0297" rpy="0 0 ${1/4*pi}"/>
   </xacro:leg>
   <!-- Leg -->
-  <xacro:leg parent="base_link" prefix="top_right">
+  <xacro:leg parent="base_link" position="top" side="right">
     <origin xyz="0.075633 -0.046741 0.0297" rpy="0 0 ${(1+1/4)*pi}"/>
   </xacro:leg>
   <!-- Leg -->
-  <xacro:leg parent="base_link" prefix="mid_right">
+  <xacro:leg parent="base_link" position="mid" side="right">
     <origin xyz="0.003574 -0.054899 0.0306" rpy="0 0 ${1*pi}"/>
   </xacro:leg>
   <!-- Leg -->
-  <xacro:leg parent="base_link" prefix="bottom_right">
+  <xacro:leg parent="base_link" position="bottom" side="right">
     <origin xyz="-0.067095 -0.046741 0.0297" rpy="0 0 ${(1-1/4)*pi}"/>
   </xacro:leg>

File: src/hexapod_description/robots/parts/arm/arm.urdf.xacro (robot description, xacro)
@@ -40,12 +40,12 @@
         <origin xyz="-0.025676 -0.000576 -0.07485" rpy="0 0 0"/>
         <geometry>
-          <mesh filename="${meshes}/arm/rotator.stl" scale="0.001 0.001 0.001"/>
+          <mesh filename="${meshes}/visual/rotator.stl" scale="0.001 0.001 0.001"/>
         </geometry>
-        <material name="dark"/>
+        <material name="PLA"/>
       </visual>
       <collision>
         <origin xyz="-0.025676 -0.000576 -0.07485" rpy="0 0 0"/>
         <geometry>
-          <mesh filename="${meshes}/arm/rotator.stl" scale="0.001 0.001 0.001"/>
+          <mesh filename="${meshes}/collision/rotator.stl" scale="0.001 0.001 0.001"/>
         </geometry>
       </collision>
@@ -60,12 +60,12 @@
         <origin xyz="-0.040258 -0.001266 -0.088773" rpy="0 0 0"/>
         <geometry>
-          <mesh filename="${meshes}/arm/abductor.stl" scale="0.001 0.001 0.001"/>
+          <mesh filename="${meshes}/visual/abductor.stl" scale="0.001 0.001 0.001"/>
         </geometry>
-        <material name="dark"/>
+        <material name="PLA"/>
       </visual>
       <collision>
         <origin xyz="-0.040258 -0.001266 -0.088773" rpy="0 0 0"/>
         <geometry>
-          <mesh filename="${meshes}/arm/abductor.stl" scale="0.001 0.001 0.001"/>
+          <mesh filename="${meshes}/collision/abductor.stl" scale="0.001 0.001 0.001"/>
         </geometry>
       </collision>
@@ -80,12 +80,12 @@
         <origin xyz="-0.039857 -0.001266 -0.135482" rpy="0 0 0"/>
         <geometry>
-          <mesh filename="${meshes}/arm/retractor.stl" scale="0.001 0.001 0.001"/>
+          <mesh filename="${meshes}/visual/retractor.stl" scale="0.001 0.001 0.001"/>
         </geometry>
-        <material name="dark"/>
+        <material name="PLA"/>
       </visual>
       <collision>
         <origin xyz="-0.039857 -0.001266 -0.135482" rpy="0 0 0"/>
         <geometry>
-          <mesh filename="${meshes}/arm/retractor.stl" scale="0.001 0.001 0.001"/>
+          <mesh filename="${meshes}/collision/retractor.stl" scale="0.001 0.001 0.001"/>
         </geometry>
       </collision>
@@ -100,12 +100,12 @@
         <origin xyz="-0.025588 0.019423 -0.0449" rpy="0 0 0"/>
         <geometry>
-          <mesh filename="${meshes}/arm/base.stl" scale="0.001 0.001 0.001"/>
+          <mesh filename="${meshes}/visual/base.stl" scale="0.001 0.001 0.001"/>
         </geometry>
-        <material name="dark"/>
+        <material name="PLA"/>
       </visual>
       <collision>
         <origin xyz="-0.025588 0.019423 -0.0449" rpy="0 0 0"/>
         <geometry>
-          <mesh filename="${meshes}/arm/base.stl" scale="0.001 0.001 0.001"/>
+          <mesh filename="${meshes}/collision/base.stl" scale="0.001 0.001 0.001"/>
         </geometry>
       </collision>

File: src/hexapod_description/robots/parts/base/base.urdf.xacro (robot description, xacro)
@@ -18,12 +18,12 @@
         <origin xyz="0 0 0" rpy="0 0 0"/>
         <geometry>
-          <mesh filename="${meshes}/base/base_link.stl" scale="0.001 0.001 0.001"/>
+          <mesh filename="${meshes}/visual/base_link.stl" scale="0.001 0.001 0.001"/>
         </geometry>
-        <material name="dark"/>
+        <material name="PLA"/>
       </visual>
       <collision>
         <origin xyz="0 0 0" rpy="0 0 0"/>
         <geometry>
-          <mesh filename="${meshes}/base/base_link.stl" scale="0.001 0.001 0.001"/>
+          <mesh filename="${meshes}/collision/base_link.stl" scale="0.001 0.001 0.001"/>
         </geometry>
       </collision>

File: src/hexapod_description/robots/parts/leg/leg.urdf.xacro (robot description, xacro)
@@ -1,33 +1,33 @@
 <?xml version="1.0"?>
 <robot xmlns:xacro="http://ros.org/wiki/xacro">
-  <xacro:macro name="leg" params="parent prefix *joint_origin">
+  <xacro:macro name="leg" params="parent position side *joint_origin">
     <!-- Joints -->
-    <joint name="${prefix}_rotate_joint" type="revolute">
+    <joint name="${position}_${side}_rotate_joint" type="revolute">
       <xacro:insert_block name="joint_origin"/>
       <parent link="${parent}"/>
-      <child link="${prefix}_cox"/>
+      <child link="${position}_${side}_cox"/>
       <axis xyz="-0.0 0.0 -1.0"/>
       <limit upper="1.570796" lower="-1.570796" effort="100" velocity="100"/>
     </joint>
-    <joint name="${prefix}_abduct_joint" type="revolute">
-      <origin xyz="0.020937 0.03 -0.021804" rpy="0 0 0"/>
+    <joint name="${position}_${side}_abduct_joint" type="revolute">
+      <origin xyz="${'0.020937 0.03 -0.021804' if side == 'left' else '0.00775 0.03 -0.021804'}" rpy="0 0 0"/>
       <axis xyz="-1.0 -0.0 -0.0"/>
       <limit upper="1.570796" lower="-1.570796" effort="100" velocity="100"/>
-      <parent link="${prefix}_cox"/>
-      <child link="${prefix}_femur"/>
+      <parent link="${position}_${side}_cox"/>
+      <child link="${position}_${side}_femur"/>
     </joint>
-    <joint name="${prefix}_retract_joint" type="revolute">
+    <joint name="${position}_${side}_retract_joint" type="revolute">
       <origin xyz="-0.029923 0.039696 -0.018563" rpy="0 0 0"/>
-      <parent link="${prefix}_femur"/>
-      <child link="${prefix}_tibia"/>
+      <parent link="${position}_${side}_femur"/>
+      <child link="${position}_${side}_tibia"/>
       <axis xyz="1.0 0.00011 0.0"/>
       <limit upper="1.570796" lower="-1.570796" effort="100" velocity="100"/>
     </joint>
-    <joint name="${prefix}_foot_joint" type="fixed">
-      <origin xyz="0.016 0.0 -0.07" rpy="0 0 0"/>
-      <parent link="${prefix}_tibia"/>
-      <child link="${prefix}_foot"/>
+    <joint name="${position}_${side}_foot_joint" type="fixed">
+      <origin xyz="0.016 0.0 -0.07"  rpi="${'0 0 ' + str(pi/2) if side == 'left' else '0 0 0'}"/>
+      <parent link="${position}_${side}_tibia"/>
+      <child link="${position}_${side}_foot"/>
     </joint>
-    <link name="${prefix}_cox">
+    <link name="${position}_${side}_cox">
       <inertial>
         <origin xyz="0.0012733261090569089 0.014903434394979126 -0.02034582182041162" rpy="0 0 0"/>
@@ -36,18 +36,19 @@
       </inertial>
       <visual>
-        <origin xyz="-0.003612 -0.056729 -0.0306" rpy="0 0 0"/>
+        <origin xyz="${'-0.003612 -0.056729 -0.0306' if side =='left' else '0.0035 -0.055 -0.0306'}"
+          rpy="${'0.0 0.0 0.0' if side == 'left' else '0.0 0.0 ' + str(pi) }"/>
         <geometry>
-          <mesh filename="${meshes}/leg/cox_left_mid.stl" scale="0.001 0.001 0.001"/>
+          <mesh filename="${meshes}/visual/cox_${side}.stl" scale="0.001 0.001 0.001"/>
         </geometry>
-        <material name="dark"/>
+        <material name="PLA"/>
       </visual>
       <collision>
         <origin xyz="-0.003612 -0.056729 -0.0306" rpy="0 0 0"/>
         <geometry>
-          <mesh filename="${meshes}/leg/cox_left_mid.stl" scale="0.001 0.001 0.001"/>
+          <mesh filename="${meshes}/collision/cox_${side}.stl" scale="0.001 0.001 0.001"/>
         </geometry>
       </collision>
     </link>
-    <link name="${prefix}_tibia">
+    <link name="${position}_${side}_tibia">
       <inertial>
         <origin xyz="0.015589179677926173 0.010695585608516162 -0.0223992522730315" rpy="0 0 0"/>
@@ -56,18 +57,19 @@
       </inertial>
       <visual>
-        <origin xyz="0.005374 -0.126425 0.009767" rpy="0 0 0"/>
+        <origin xyz="${'0.005374 -0.126425 0.009767' if side == 'left' else '0.0275 -0.125 0.01'}"
+          rpy="0 0 ${0 if side =='left' else pi}"/>
         <geometry>
-          <mesh filename="${meshes}/leg/tibia_left_mid.stl" scale="0.001 0.001 0.001"/>
+          <mesh filename="${meshes}/visual/tibia_${side}.stl" scale="0.001 0.001 0.001"/>
         </geometry>
-        <material name="dark"/>
+        <material name="PLA"/>
       </visual>
       <collision>
         <origin xyz="0.005374 -0.126425 0.009767" rpy="0 0 0"/>
         <geometry>
-          <mesh filename="${meshes}/leg/tibia_left_mid.stl" scale="0.001 0.001 0.001"/>
+          <mesh filename="${meshes}/collision/tibia_${side}.stl" scale="0.001 0.001 0.001"/>
         </geometry>
       </collision>
     </link>
-    <link name="${prefix}_foot">
+    <link name="${position}_${side}_foot">
       <visual>
         <origin xyz="0.0 0.0 0.0" rpy="0 0 0"/>
@@ -75,8 +77,8 @@
           <sphere  radius="0.0080"/>
         </geometry>
-        <material name="dark"/>
+        <material name="TPU"/>
       </visual>
     </link>
-    <link name="${prefix}_femur">
+    <link name="${position}_${side}_femur">
       <inertial>
         <origin xyz="-0.015011654934717145 0.020989624323966824 -0.005728252734904802" rpy="0 0 0"/>
@@ -85,43 +87,44 @@
       </inertial>
       <visual>
-        <origin xyz="-0.024549 -0.086729 -0.008796" rpy="0 0 0"/>
+        <origin xyz="${'-0.024549 -0.086729 -0.008796' if side == 'left' else '-0.0035 -0.085 -0.0085'}"
+          rpy="0.0 0.0 ${0 if side =='left' else pi}"/>
         <geometry>
-          <mesh filename="${meshes}/leg/femur_left_mid.stl" scale="0.001 0.001 0.001"/>
+          <mesh filename="${meshes}/visual/femur_${side}.stl" scale="0.001 0.001 0.001"/>
         </geometry>
-        <material name="dark"/>
+        <material name="PLA"/>
       </visual>
       <collision>
         <origin xyz="-0.024549 -0.086729 -0.008796" rpy="0 0 0"/>
         <geometry>
-          <mesh filename="${meshes}/leg/femur_left_mid.stl" scale="0.001 0.001 0.001"/>
+          <mesh filename="${meshes}/collision/femur_${side}.stl" scale="0.001 0.001 0.001"/>
         </geometry>
       </collision>
     </link>
-    <transmission name="${prefix}_rotate_joint_tran">
+    <transmission name="${position}_${side}_rotate_joint_tran">
       <type>transmission_interface/SimpleTransmission</type>
-      <joint name="${prefix}_rotate_joint">
+      <joint name="${position}_${side}_rotate_joint">
         <hardwareInterface>hardware_interface/EffortJointInterface</hardwareInterface>
       </joint>
-      <actuator name="${prefix}_rotate_joint_actr">
+      <actuator name="${position}_${side}_rotate_joint_actr">
         <hardwareInterface>hardware_interface/EffortJointInterface</hardwareInterface>
         <mechanicalReduction>1</mechanicalReduction>
       </actuator>
     </transmission>
-    <transmission name="${prefix}_abduct_joint_tran">
+    <transmission name="${position}_${side}_abduct_joint_tran">
       <type>transmission_interface/SimpleTransmission</type>
-      <joint name="${prefix}_abduct_joint">
+      <joint name="${position}_${side}_abduct_joint">
         <hardwareInterface>hardware_interface/EffortJointInterface</hardwareInterface>
       </joint>
-      <actuator name="${prefix}_abduct_joint_actr">
+      <actuator name="${position}_${side}_abduct_joint_actr">
         <hardwareInterface>hardware_interface/EffortJointInterface</hardwareInterface>
         <mechanicalReduction>1</mechanicalReduction>
       </actuator>
     </transmission>
-    <transmission name="${prefix}_retract_joint_tran">
+    <transmission name="${position}_${side}_retract_joint_tran">
       <type>transmission_interface/SimpleTransmission</type>
-      <joint name="${prefix}_retract_joint">
+      <joint name="${position}_${side}_retract_joint">
         <hardwareInterface>hardware_interface/EffortJointInterface</hardwareInterface>
       </joint>
-      <actuator name="${prefix}_retract_joint_actr">
+      <actuator name="${position}_${side}_retract_joint_actr">
         <hardwareInterface>hardware_interface/EffortJointInterface</hardwareInterface>
         <mechanicalReduction>1</mechanicalReduction>

File: src/hexapod_description/robots/parts/sensors/sipeed_maixsense_a010.urdf.xacro (robot description, xacro)
@@ -28,12 +28,12 @@
         <origin xyz="-0.185 -0.0275 0.0" rpy="${1/2*pi} 0 ${1/2*pi}"/>
       <geometry>
-        <mesh filename="${meshes}/sensors/camera/camera.stl" scale="0.001 0.001 0.001"/>
+        <mesh filename="${meshes}/visual/camera_case_cover.stl" scale="0.001 0.001 0.001"/>
       </geometry>
-      <material name="dark"/>
+      <material name="PLA"/>
     </visual>
       <collision>
         <origin xyz="0.041999 0.020484 -0.080935" rpy="0 0 0"/>
         <geometry>
-          <mesh filename="${meshes}/sensors/camera/camera.stl" scale="0.001 0.001 0.001"/>
+          <mesh filename="${meshes}/collision/camera_case_cover.stl" scale="0.001 0.001 0.001"/>
         </geometry>
       </collision>
@@ -42,5 +42,5 @@
     <link name="depth_camera_link">
     <visual>
-        <origin xyz="0.0 0.0025 0.0" rpy="0 0 0"/>
+        <origin xyz="-0.0125 0.0025 -0.0" rpy="0 0 0"/>
       <geometry>
         <box size="0.01 0.04 0.03"/>

Commit message: Inverse kinematics works for all joints

File: src/hexapod_description/materials/hexapod.materials.xacro (robot description, xacro)
@@ -4,5 +4,5 @@
   <!-- Init colour -->
   <material name="TPU">
-    <color rgba="0.0 0.0 0.0 1.0"/>
+    <color rgba="0.3 0.3 0.3 1.0"/>
   </material>
   <material name="PLA">

File: src/hexapod_description/robots/parts/leg/leg.urdf.xacro (robot description, xacro)
@@ -44,5 +44,6 @@
       </visual>
       <collision>
-        <origin xyz="-0.003612 -0.056729 -0.0306" rpy="0 0 0"/>
+        <origin xyz="${'-0.003612 -0.056729 -0.0306' if side =='left' else '0.0035 -0.055 -0.0306'}"
+          rpy="${'0.0 0.0 0.0' if side == 'left' else '0.0 0.0 ' + str(pi) }"/>
         <geometry>
           <mesh filename="${meshes}/collision/cox_${side}.stl" scale="0.001 0.001 0.001"/>
@@ -65,5 +66,6 @@
       </visual>
       <collision>
-        <origin xyz="0.005374 -0.126425 0.009767" rpy="0 0 0"/>
+        <origin xyz="${'0.005374 -0.126425 0.009767' if side == 'left' else '0.0275 -0.125 0.01'}"
+          rpy="0 0 ${0 if side =='left' else pi}"/>
         <geometry>
           <mesh filename="${meshes}/collision/tibia_${side}.stl" scale="0.001 0.001 0.001"/>
@@ -95,5 +97,6 @@
       </visual>
       <collision>
-        <origin xyz="-0.024549 -0.086729 -0.008796" rpy="0 0 0"/>
+        <origin xyz="${'-0.024549 -0.086729 -0.008796' if side == 'left' else '-0.0035 -0.085 -0.0085'}"
+          rpy="0.0 0.0 ${0 if side =='left' else pi}"/>
         <geometry>
           <mesh filename="${meshes}/collision/femur_${side}.stl" scale="0.001 0.001 0.001"/>
