Commit message: Seperated launch files into reusable launch files

File: hexapod.urdf (robot description, URDF)
Before this commit: robot hexapod, 33 links, 32 joints
Links:
- link bottom_left_foot: mass None -> 0.01; geometry collision sphere radius=0.0080; visual sphere radius=0.0080
- link bottom_right_foot: mass None -> 0.01; geometry collision sphere radius=0.0080; visual sphere radius=0.0080
- link mid_left_foot: mass None -> 0.01; geometry collision sphere radius=0.0080; visual sphere radius=0.0080
- link mid_right_foot: mass None -> 0.01; geometry collision sphere radius=0.0080; visual sphere radius=0.0080
- link top_left_foot: mass None -> 0.01; geometry collision sphere radius=0.0080; visual sphere radius=0.0080
- link top_right_foot: mass None -> 0.01; geometry collision sphere radius=0.0080; visual sphere radius=0.0080

File: src/hexapod_description/robots/parts/leg/leg.urdf.xacro (robot description, xacro)
@@ -73,13 +73,50 @@
       </collision>
     </link>
-    <link name="${position}_${side}_foot">
-      <visual>
-        <origin xyz="0.0 0.0 0.0" rpy="0 0 0"/>
-        <geometry>
-          <sphere  radius="0.0080"/>
-        </geometry>
-        <material name="TPU"/>
-      </visual>
-    </link>
+<link name="${position}_${side}_foot">
+<inertial>
+    <origin xyz="0 0 0" rpy="0 0 0"/>
+    <mass value="0.01"/>
+    <inertia
+      ixx="1.28e-6" ixy="0" ixz="0"
+      iyy="1.28e-6" iyz="0"
+      izz="1.28e-6"/>
+  </inertial>
+  <collision name="foot_collision">
+    <origin xyz="0.0 0.0 0.0" rpy="0 0 0"/>
+    <geometry>
+      <sphere radius="0.0080"/>
+    </geometry>
+ <surface>
+    <friction>
+      <ode>
+        <mu>1000000.0</mu>     <!-- Max static friction -->
+        <mu2>1000000.0</mu2>   <!-- Max dynamic friction -->
+      </ode>
+    </friction>
+    <contact>
+      <ode>
+        <kp>100000</kp>       <!-- stiffness -->
+        <kd>100</kd>          <!-- damping -->
+        <max_vel>0.1</max_vel>
+        <min_depth>0.001</min_depth>
+      </ode>
+    </contact>
+  </surface>
+  </collision>
+  <visual>
+    <origin xyz="0.0 0.0 0.0" rpy="0 0 0"/>
+    <geometry>
+      <sphere radius="0.0080"/>
+    </geometry>
+    <material name="TPU"/>
+  </visual>
+</link>
+<!-- <collision name="bottom_left_femur_collision"> -->
+<!--   <geometry> -->
+<!--     <mesh> -->
+<!--       <uri>package://your_package/meshes/femur_collision.dae</uri> -->
+<!--     </mesh> -->
+<!--   </geometry> -->
+<!-- </collision> -->
     <link name="${position}_${side}_femur">
       <inertial>

File: src/hexapod_description/ros2_control/hexapod.ros2_control.xacro (robot description, xacro)
@@ -1,13 +1,5 @@
-<?xml version="1.0"?>
+<?xml version="1.0" encoding="UTF-8"?>
 <robot xmlns:xacro="http://www.ros.org/wiki/xacro">
   <xacro:macro name="joint" params="name">
-    <!-- Code to set params from .yaml file -->
-            <!-- <joint name="top_left_rotate_joint"> -->
-            <!--     <command_interface name="position"/> -->
-            <!--     <state_interface name="position"> -->
-            <!--       <param name="initial_value">${initial_positions['top_left_rotate_joint']}</param> -->
-            <!--     </state_interface> -->
-            <!--     <state_interface name="velocity"/> -->
-            <!-- </joint> -->
     <joint name="${name}">
       <command_interface name="position">
@@ -15,39 +7,47 @@
         <param name="max">1.5</param>
       </command_interface>
-      <state_interface name="position"/>
+      <state_interface name="position"></state_interface>
     </joint>
   </xacro:macro>
   <gazebo>
     <plugin filename="libgz_ros2_control-system" name="gz_ros2_control::GazeboSimROS2ControlPlugin">
-      <parameters>$(find hexapod_bringup)/config/hexapod_controllers.yaml</parameters>
+      <parameters>$(find hexapod_sim)/config/hexapod_controllers.yaml</parameters>
     </plugin>
   </gazebo>
-    <xacro:macro name="hexapod_ros2_control" params="name initial_positions_file">
-        <xacro:property name="initial_positions" value="${xacro.load_yaml(initial_positions_file)['initial_positions']}"/>
+  <!-- Code to set params from .yaml file -->
+  <!-- <joint name="top_left_rotate_joint"> -->
+  <!--     <command_interface name="position"/> -->
+  <!--     <state_interface name="position"> -->
+  <!--       <param name="initial_value">${initial_positions['top_left_rotate_joint']}</param> -->
+  <!--     </state_interface> -->
+  <!--     <state_interface name="velocity"/> -->
+  <!-- </joint> -->
+  <xacro:macro name="hexapod_ros2_control" params="name initial_positions_file">
+    <xacro:property name="initial_positions" value="${xacro.load_yaml(initial_positions_file)['initial_positions']}"></xacro:property>
     <ros2_control name="${name}" type="system">
       <hardware>
         <plugin>gz_ros2_control/GazeboSimSystem</plugin>
       </hardware>
-      <xacro:joint name="arm_rotator_joint"/>
-      <xacro:joint name="arm_abductor_joint"/>
-      <xacro:joint name="arm_retractor_joint"/>
-      <xacro:joint name="top_left_rotate_joint"/>
-      <xacro:joint name="top_left_abduct_joint"/>
-      <xacro:joint name="top_left_retract_joint"/>
-      <xacro:joint name="mid_left_rotate_joint"/>
-      <xacro:joint name="mid_left_abduct_joint"/>
-      <xacro:joint name="mid_left_retract_joint"/>
-      <xacro:joint name="bottom_left_rotate_joint"/>
-      <xacro:joint name="bottom_left_abduct_joint"/>
-      <xacro:joint name="bottom_left_retract_joint"/>
-      <xacro:joint name="top_right_rotate_joint"/>
-      <xacro:joint name="top_right_abduct_joint"/>
-      <xacro:joint name="top_right_retract_joint"/>
-      <xacro:joint name="mid_right_rotate_joint"/>
-      <xacro:joint name="mid_right_abduct_joint"/>
-      <xacro:joint name="mid_right_retract_joint"/>
-      <xacro:joint name="bottom_right_rotate_joint"/>
-      <xacro:joint name="bottom_right_abduct_joint"/>
-      <xacro:joint name="bottom_right_retract_joint"/>
+      <xacro:joint name="arm_rotator_joint"></xacro:joint>
+      <xacro:joint name="arm_abductor_joint"></xacro:joint>
+      <xacro:joint name="arm_retractor_joint"></xacro:joint>
+      <xacro:joint name="top_left_rotate_joint"></xacro:joint>
+      <xacro:joint name="top_left_abduct_joint"></xacro:joint>
+      <xacro:joint name="top_left_retract_joint"></xacro:joint>
+      <xacro:joint name="mid_left_rotate_joint"></xacro:joint>
+      <xacro:joint name="mid_left_abduct_joint"></xacro:joint>
+      <xacro:joint name="mid_left_retract_joint"></xacro:joint>
+      <xacro:joint name="bottom_left_rotate_joint"></xacro:joint>
+      <xacro:joint name="bottom_left_abduct_joint"></xacro:joint>
+      <xacro:joint name="bottom_left_retract_joint"></xacro:joint>
+      <xacro:joint name="top_right_rotate_joint"></xacro:joint>
+      <xacro:joint name="top_right_abduct_joint"></xacro:joint>
+      <xacro:joint name="top_right_retract_joint"></xacro:joint>
+      <xacro:joint name="mid_right_rotate_joint"></xacro:joint>
+      <xacro:joint name="mid_right_abduct_joint"></xacro:joint>
+      <xacro:joint name="mid_right_retract_joint"></xacro:joint>
+      <xacro:joint name="bottom_right_rotate_joint"></xacro:joint>
+      <xacro:joint name="bottom_right_abduct_joint"></xacro:joint>
+      <xacro:joint name="bottom_right_retract_joint"></xacro:joint>
     </ros2_control>
   </xacro:macro>
