Commit message: Added Joystick support, can control Arm

File: src/hexapod_description/robots/hexapod.urdf.xacro (robot description, xacro)
@@ -7,5 +7,5 @@
   <xacro:property name="meshes" value="file://$(find hexapod_description)/meshes"/>
   <xacro:include filename="$(find hexapod_description)/gazebo/hexapod.gazebo.xacro"/>
-  <!-- <xacro:include filename="$(find hexapod_description)/ros2_control/hexapod.ros2_control.xacro"/> -->
+  <xacro:include filename="$(find hexapod_description)/ros2_control/hexapod.ros2_control.xacro"/>
   <xacro:include filename="$(find hexapod_description)/materials/hexapod.materials.xacro"/>
   <xacro:include filename="${robots}/parts/base/base.urdf.xacro"/>
@@ -13,4 +13,6 @@
   <xacro:include filename="${robots}/parts/leg/leg.urdf.xacro"/>
   <xacro:include filename="${robots}/parts/camera/camera.urdf.xacro"/>
+  <!-- ================== ARGS ===================== -->
+  <xacro:arg name="initial_positions_file" default="initial_positions.yaml" />
   <!-- =============== Link & Joint =============== -->
   <!-- Base -->
@@ -55,4 +57,4 @@
   <!-- =============== Gazebo =============== -->
   <xacro:hexapod_gazebo/>
-  <!-- <xacro:hexapod_ros2_control/> -->
+  <xacro:hexapod_ros2_control name="FakeSystem" initial_positions_file="$(arg initial_positions_file)"/>
 </robot>

File: src/hexapod_description/robots/parts/arm/arm.urdf.xacro (robot description, xacro)
@@ -27,4 +27,5 @@
       <child link="arm_retractor"/>
       <axis xyz="-0.999993 0.0 -0.003676"/>
+      p
       <limit upper="1.570796" lower="-1.570796" effort="100" velocity="100"/>
     </joint>

File: src/hexapod_description/robots/parts/leg/leg.urdf.xacro (robot description, xacro)
@@ -21,5 +21,5 @@
       <parent link="${prefix}_femur"/>
       <child link="${prefix}_tibia"/>
-      <axis xyz="0.707029 0.707185 0.0"/>
+      <axis xyz="1.0 0.00011 0.0"/>
       <limit upper="1.570796" lower="-1.570796" effort="100" velocity="100"/>
     </joint>

File: src/hexapod_description/ros2_control/hexapod.ros2_control.xacro (robot description, xacro)
@@ -2,8 +2,16 @@
 <robot xmlns:xacro="http://www.ros.org/wiki/xacro">
   <xacro:macro name="joint" params="name">
+    <!-- Code to set params from .yaml file -->
+            <!-- <joint name="top_left_rotate_joint"> -->
+            <!--     <command_interface name="position"/> -->
+            <!--     <state_interface name="position"> -->
+            <!--       <param name="initial_value">${initial_positions['top_left_rotate_joint']}</param> -->
+            <!--     </state_interface> -->
+            <!--     <state_interface name="velocity"/> -->
+            <!-- </joint> -->
     <joint name="${name}">
       <command_interface name="position">
-        <param name="min">-1</param>
-        <param name="max">1</param>
+        <param name="min">-1.5</param>
+        <param name="max">1.5</param>
       </command_interface>
       <state_interface name="position"/>
@@ -15,6 +23,7 @@
     </plugin>
   </gazebo>
-  <xacro:macro name="hexapod_ros2_control">
-    <ros2_control name="GazeboSystem" type="system">
+    <xacro:macro name="hexapod_ros2_control" params="name initial_positions_file">
+        <xacro:property name="initial_positions" value="${xacro.load_yaml(initial_positions_file)['initial_positions']}"/>
+    <ros2_control name="${name}" type="system">
       <hardware>
         <plugin>gz_ros2_control/GazeboSimSystem</plugin>

File: src/hexapod_moveit/config/hexapod.ros2_control.xacro (robot description, xacro)
@@ -29,4 +29,130 @@
                 <state_interface name="velocity"/>
             </joint>
+            <joint name="top_left_rotate_joint">
+                <command_interface name="position"/>
+                <state_interface name="position">
+                  <param name="initial_value">${initial_positions['top_left_rotate_joint']}</param>
+                </state_interface>
+                <state_interface name="velocity"/>
+            </joint>
+            <joint name="top_left_abduct_joint">
+                <command_interface name="position"/>
+                <state_interface name="position">
+                  <param name="initial_value">${initial_positions['top_left_abduct_joint']}</param>
+                </state_interface>
+                <state_interface name="velocity"/>
+            </joint>
+            <joint name="top_left_retract_joint">
+                <command_interface name="position"/>
+                <state_interface name="position">
+                  <param name="initial_value">${initial_positions['top_left_retract_joint']}</param>
+                </state_interface>
+                <state_interface name="velocity"/>
+            </joint>
+            <joint name="mid_left_rotate_joint">
+                <command_interface name="position"/>
+                <state_interface name="position">
+                  <param name="initial_value">${initial_positions['mid_left_rotate_joint']}</param>
+                </state_interface>
+                <state_interface name="velocity"/>
+            </joint>
+            <joint name="mid_left_abduct_joint">
+                <command_interface name="position"/>
+                <state_interface name="position">
+                  <param name="initial_value">${initial_positions['mid_left_abduct_joint']}</param>
+                </state_interface>
+                <state_interface name="velocity"/>
+            </joint>
+            <joint name="mid_left_retract_joint">
+                <command_interface name="position"/>
+                <state_interface name="position">
+                  <param name="initial_value">${initial_positions['mid_left_retract_joint']}</param>
+                </state_interface>
+                <state_interface name="velocity"/>
+            </joint>
+            <joint name="bottom_left_rotate_joint">
+                <command_interface name="position"/>
+                <state_interface name="position">
+                  <param name="initial_value">${initial_positions['bottom_left_rotate_joint']}</param>
+                </state_interface>
+                <state_interface name="velocity"/>
+            </joint>
+            <joint name="bottom_left_abduct_joint">
+                <command_interface name="position"/>
+                <state_interface name="position">
+                  <param name="initial_value">${initial_positions['bottom_left_abduct_joint']}</param>
+                </state_interface>
+                <state_interface name="velocity"/>
+            </joint>
+            <joint name="bottom_left_retract_joint">
+                <command_interface name="position"/>
+                <state_interface name="position">
+                  <param name="initial_value">${initial_positions['bottom_left_retract_joint']}</param>
+                </state_interface>
+                <state_interface name="velocity"/>
+            </joint>
+            <joint name="top_right_rotate_joint">
+                <command_interface name="position"/>
+                <state_interface name="position">
+                  <param name="initial_value">${initial_positions['top_right_rotate_joint']}</param>
+                </state_interface>
+                <state_interface name="velocity"/>
+            </joint>
+            <joint name="top_right_abduct_joint">
+                <command_interface name="position"/>
+                <state_interface name="position">
+                  <param name="initial_value">${initial_positions['top_right_abduct_joint']}</param>
+                </state_interface>
+                <state_interface name="velocity"/>
+            </joint>
+            <joint name="top_right_retract_joint">
+                <command_interface name="position"/>
+                <state_interface name="position">
+                  <param name="initial_value">${initial_positions['top_right_retract_joint']}</param>
+                </state_interface>
+                <state_interface name="velocity"/>
+            </joint>
+            <joint name="mid_right_rotate_joint">
+                <command_interface name="position"/>
+                <state_interface name="position">
+                  <param name="initial_value">${initial_positions['mid_right_rotate_joint']}</param>
+                </state_interface>
+                <state_interface name="velocity"/>
+            </joint>
+            <joint name="mid_right_abduct_joint">
+                <command_interface name="position"/>
+                <state_interface name="position">
+                  <param name="initial_value">${initial_positions['mid_right_abduct_joint']}</param>
+                </state_interface>
+                <state_interface name="velocity"/>
+            </joint>
+            <joint name="mid_right_retract_joint">
+                <command_interface name="position"/>
+                <state_interface name="position">
+                  <param name="initial_value">${initial_positions['mid_right_retract_joint']}</param>
+                </state_interface>
+                <state_interface name="velocity"/>
+            </joint>
+            <joint name="bottom_right_rotate_joint">
+                <command_interface name="position"/>
+                <state_interface name="position">
+                  <param name="initial_value">${initial_positions['bottom_right_rotate_joint']}</param>
+                </state_interface>
+                <state_interface name="velocity"/>
+            </joint>
+            <joint name="bottom_right_abduct_joint">
+                <command_interface name="position"/>
+                <state_interface name="position">
+                  <param name="initial_value">${initial_positions['bottom_right_abduct_joint']}</param>
+                </state_interface>
+                <state_interface name="velocity"/>
+            </joint>
+            <joint name="bottom_right_retract_joint">
+                <command_interface name="position"/>
+                <state_interface name="position">
+                  <param name="initial_value">${initial_positions['bottom_right_retract_joint']}</param>
+                </state_interface>
+                <state_interface name="velocity"/>
+            </joint>
         </ros2_control>
     </xacro:macro>

Commit message: Arm Control Panel works

File: src/hexapod_description/robots/hexapod.urdf.xacro (robot description, xacro)
@@ -29,5 +29,5 @@
   <!-- Camera -->
   <xacro:camera parent="arm_retractor">
-    <origin xyz="-0.081856 -0.02175 -0.054547" rpy="0 0 0"/>
+    <origin xyz="-0.0125 0.0 0.05" rpy="0 ${-1/2*M_PI} 0"/>
   </xacro:camera>
   <!-- Leg -->

File: src/hexapod_description/robots/parts/camera/camera.urdf.xacro (robot description, xacro)
@@ -20,5 +20,5 @@
       </inertial>
       <visual>
-        <origin xyz="0.041999 0.020484 -0.080935" rpy="0 0 0"/>
+        <origin xyz="-0.18 0.0 0.0285" rpy="0 ${1/2*M_PI} 0"/>
         <geometry>
           <mesh filename="${meshes}/sensors/camera/camera.stl" scale="0.001 0.001 0.001"/>

Commit message: Fixed Camera

File: src/hexapod_description/robots/hexapod.urdf.xacro (robot description, xacro)
@@ -29,5 +29,5 @@
   <!-- Camera -->
   <xacro:camera parent="arm_retractor">
-    <origin xyz="-0.0125 0.0 0.05" rpy="0 ${-1/2*M_PI} 0"/>
+    <origin xyz="-0.0125 0.0 0.055" rpy="0 ${-1/2*M_PI} ${-1/2*M_PI}"/>
   </xacro:camera>
   <!-- Leg -->

File: src/hexapod_description/robots/parts/camera/camera.urdf.xacro (robot description, xacro)
@@ -10,8 +10,14 @@
       <xacro:insert_block name="joint_origin"/>
       <parent link="${parent}"/>
+      <child link="camera_case_cover"/>
+    </joint>
+    <!-- Joints -->
+    <joint name="camera_mount" type="fixed">
+      <xacro:insert_block name="joint_origin"/>
+      <parent link="${parent}"/>
       <child link="camera_link"/>
     </joint>
     <!-- Links -->
-    <link name="camera_link">
+    <link name="camera_case_cover">
       <inertial>
         <origin xyz="0.07257325961305607 0.023187735063927437 0.09454807900867684" rpy="0 0 0"/>
@@ -19,11 +25,11 @@
         <inertia ixx="1e-06" iyy="2e-06" izz="3e-06" ixy="0.0" iyz="0.0" ixz="0.0"/>
       </inertial>
-      <visual>
-        <origin xyz="-0.18 0.0 0.0285" rpy="0 ${1/2*M_PI} 0"/>
-        <geometry>
-          <mesh filename="${meshes}/sensors/camera/camera.stl" scale="0.001 0.001 0.001"/>
-        </geometry>
-        <material name="dark"/>
-      </visual>
+    <visual>
+        <origin xyz="-0.185 -0.0275 0.0" rpy="${1/2*M_PI} 0 ${1/2*M_PI}"/>
+      <geometry>
+        <mesh filename="${meshes}/sensors/camera/camera.stl" scale="0.001 0.001 0.001"/>
+      </geometry>
+      <material name="dark"/>
+    </visual>
       <collision>
         <origin xyz="0.041999 0.020484 -0.080935" rpy="0 0 0"/>
@@ -32,4 +38,7 @@
         </geometry>
       </collision>
+    </link>
+    <!-- Links -->
+    <link name="camera_link">
     </link>
     <!-- Gazebo -->

Commit message: Added points in Rviz

File: src/hexapod_description/robots/hexapod.urdf.xacro (robot description, xacro)
@@ -21,5 +21,5 @@
   <!-- Base -->
   <xacro:base parent="base_footprint">
-    <origin xyz="0 0 0.8" rpy="0 0 0"/>
+    <origin xyz="0 0 0.4" rpy="0 0 0"/>
   </xacro:base>
   <!-- Arm -->
@@ -27,8 +27,4 @@
     <origin xyz="0.025588 -0.019423 0.0449" rpy="0 0 0"/>
   </xacro:arm>
-  <!-- Camera -->
-  <xacro:camera parent="arm_retractor">
-    <origin xyz="-0.0125 0.0 0.055" rpy="0 ${-1/2*M_PI} ${-1/2*M_PI}"/>
-  </xacro:camera>
   <!-- Leg -->
   <xacro:leg parent="base_link" prefix="top_left">
@@ -55,4 +51,8 @@
     <origin xyz="-0.067095 -0.046741 0.0297" rpy="0 0 ${(1-1/4)*M_PI}"/>
   </xacro:leg>
+  <!-- ================ Camera =============== -->
+  <xacro:camera parent="arm_retractor">
+    <origin xyz="-0.0125 0.0 0.055" rpy="0 ${-1/2*M_PI} ${-1/2*M_PI}"/>
+  </xacro:camera>
   <!-- =============== Gazebo =============== -->
   <xacro:hexapod_gazebo/>

File: src/hexapod_description/robots/parts/camera/camera.urdf.xacro (robot description, xacro)
@@ -7,47 +7,48 @@
   <xacro:macro name="camera" params="parent *joint_origin">
     <!-- Joints -->
-    <joint name="camera_case_mount" type="fixed">
-      <xacro:insert_block name="joint_origin"/>
-      <parent link="${parent}"/>
-      <child link="camera_case_cover"/>
-    </joint>
+    <!-- <joint name="camera_case_mount" type="fixed"> -->
+    <!--   <xacro:insert_block name="joint_origin"/> -->
+    <!--   <parent link="${parent}"/> -->
+    <!--   <child link="camera_case_cover"/> -->
+    <!-- </joint> -->
     <!-- Joints -->
     <joint name="camera_mount" type="fixed">
       <xacro:insert_block name="joint_origin"/>
       <parent link="${parent}"/>
-      <child link="camera_link"/>
+      <child link="depth_camera_link"/>
     </joint>
     <!-- Links -->
-    <link name="camera_case_cover">
-      <inertial>
-        <origin xyz="0.07257325961305607 0.023187735063927437 0.09454807900867684" rpy="0 0 0"/>
-        <mass value="0.00672643608404174"/>
-        <inertia ixx="1e-06" iyy="2e-06" izz="3e-06" ixy="0.0" iyz="0.0" ixz="0.0"/>
-      </inertial>
-    <visual>
-        <origin xyz="-0.185 -0.0275 0.0" rpy="${1/2*M_PI} 0 ${1/2*M_PI}"/>
-      <geometry>
-        <mesh filename="${meshes}/sensors/camera/camera.stl" scale="0.001 0.001 0.001"/>
-      </geometry>
-      <material name="dark"/>
-    </visual>
-      <collision>
-        <origin xyz="0.041999 0.020484 -0.080935" rpy="0 0 0"/>
-        <geometry>
-          <mesh filename="${meshes}/sensors/camera/camera.stl" scale="0.001 0.001 0.001"/>
-        </geometry>
-      </collision>
-    </link>
+    <!-- <link name="camera_case_cover"> -->
+    <!--   <inertial> -->
+    <!--     <origin xyz="0.07257325961305607 0.023187735063927437 0.09454807900867684" rpy="0 0 0"/> -->
+    <!--     <mass value="0.00672643608404174"/> -->
+    <!--     <inertia ixx="1e-06" iyy="2e-06" izz="3e-06" ixy="0.0" iyz="0.0" ixz="0.0"/> -->
+    <!--   </inertial> -->
+    <!-- <visual> -->
+    <!--     <origin xyz="-0.185 -0.0275 0.0" rpy="${1/2*M_PI} 0 ${1/2*M_PI}"/> -->
+    <!--   <geometry> -->
+    <!--     <mesh filename="${meshes}/sensors/camera/camera.stl" scale="0.001 0.001 0.001"/> -->
+    <!--   </geometry> -->
+    <!--   <material name="dark"/> -->
+    <!-- </visual> -->
+    <!--   <collision> -->
+    <!--     <origin xyz="0.041999 0.020484 -0.080935" rpy="0 0 0"/> -->
+    <!--     <geometry> -->
+    <!--       <mesh filename="${meshes}/sensors/camera/camera.stl" scale="0.001 0.001 0.001"/> -->
+    <!--     </geometry> -->
+    <!--   </collision> -->
+    <!-- </link> -->
+    <!---->
     <!-- Links -->
-    <link name="camera_link">
+    <link name="depth_camera_link">
     </link>
     <!-- Gazebo -->
-    <gazebo reference="camera_link">
-      <sensor name="depth_camera" type="depth_camera">
+    <gazebo reference="depth_camera_link">
+      <sensor name="depth_camera_link" type="depth_camera">
         <always_on>true</always_on>
         <visualize>true</visualize>
         <update_rate>60</update_rate>
         <topic>depth_camera/depth/image_raw</topic>
-        <frame_id>camera_depth_frame</frame_id>
+        <frame_id>hexapod/arm_retractor/depth_camera_link</frame_id>
         <camera name="Sipeed MaixSense A10">
           <camera_info_topic>depth_camera/depth/camera_info</camera_info_topic>

Commit message: Increased controller update rate

File: src/hexapod_description/robots/hexapod.urdf.xacro (robot description, xacro)
@@ -2,5 +2,4 @@
 <!-- Basic differential drive mobile base -->
 <robot xmlns:xacro="http://www.ros.org/wiki/xacro" name="hexapod">
-  <xacro:property name="M_PI" value="3.14159274"/>
   <xacro:property name="description_package" value="$(find hexapod_description)"/>
   <xacro:property name="robots" value="${description_package}/robots"/>
@@ -12,5 +11,5 @@
   <xacro:include filename="${robots}/parts/arm/arm.urdf.xacro"/>
   <xacro:include filename="${robots}/parts/leg/leg.urdf.xacro"/>
-  <xacro:include filename="${robots}/parts/camera/camera.urdf.xacro"/>
+  <xacro:include filename="${robots}/parts/sensors/sipeed_maixsense_a010.urdf.xacro"/>
   <!-- ================== ARGS ===================== -->
   <xacro:arg name="initial_positions_file" default="initial_positions.yaml" />
@@ -29,5 +28,5 @@
   <!-- Leg -->
   <xacro:leg parent="base_link" prefix="top_left">
-    <origin xyz="0.074451 0.046824 0.0297" rpy="0 0 ${-1/4*M_PI}"/>
+    <origin xyz="0.074451 0.046824 0.0297" rpy="0 0 ${-1/4*pi}"/>
   </xacro:leg>
   <!-- Leg -->
@@ -37,21 +36,21 @@
   <!-- Leg -->
   <xacro:leg parent="base_link" prefix="bottom_left">
-    <origin xyz="-0.067095 0.047401 0.0297" rpy="0 0 ${1/4*M_PI}"/>
+    <origin xyz="-0.067095 0.047401 0.0297" rpy="0 0 ${1/4*pi}"/>
   </xacro:leg>
   <!-- Leg -->
   <xacro:leg parent="base_link" prefix="top_right">
-    <origin xyz="0.075633 -0.046741 0.0297" rpy="0 0 ${(1+1/4)*M_PI}"/>
+    <origin xyz="0.075633 -0.046741 0.0297" rpy="0 0 ${(1+1/4)*pi}"/>
   </xacro:leg>
   <!-- Leg -->
   <xacro:leg parent="base_link" prefix="mid_right">
-    <origin xyz="0.003574 -0.054899 0.0306" rpy="0 0 ${1*M_PI}"/>
+    <origin xyz="0.003574 -0.054899 0.0306" rpy="0 0 ${1*pi}"/>
   </xacro:leg>
   <!-- Leg -->
   <xacro:leg parent="base_link" prefix="bottom_right">
-    <origin xyz="-0.067095 -0.046741 0.0297" rpy="0 0 ${(1-1/4)*M_PI}"/>
+    <origin xyz="-0.067095 -0.046741 0.0297" rpy="0 0 ${(1-1/4)*pi}"/>
   </xacro:leg>
   <!-- ================ Camera =============== -->
   <xacro:camera parent="arm_retractor">
-    <origin xyz="-0.0125 0.0 0.055" rpy="0 ${-1/2*M_PI} ${-1/2*M_PI}"/>
+    <origin xyz="-0.0125 0.0 0.055" rpy="0 ${-1/2*pi} ${-1/2*pi}"/>
   </xacro:camera>
   <!-- =============== Gazebo =============== -->

File: src/hexapod_description/robots/parts/sensors/sipeed_maixsense_a010.urdf.xacro (robot description, xacro)
@@ -26,5 +26,5 @@
       </inertial>
     <visual>
-        <origin xyz="-0.185 -0.0275 0.0" rpy="${1/2*M_PI} 0 ${1/2*M_PI}"/>
+        <origin xyz="-0.185 -0.0275 0.0" rpy="${1/2*pi} 0 ${1/2*pi}"/>
       <geometry>
         <mesh filename="${meshes}/sensors/camera/camera.stl" scale="0.001 0.001 0.001"/>

Commit message: Updated Rviz config file

File: src/hexapod_description/robots/hexapod.urdf.xacro (robot description, xacro)
@@ -3,4 +3,5 @@
 <robot xmlns:xacro="http://www.ros.org/wiki/xacro" name="hexapod">
   <xacro:property name="description_package" value="$(find hexapod_description)"/>
+  <xacro:property name="HEXAPOD_HEIGHT" value="0.085"/>
   <xacro:property name="robots" value="${description_package}/robots"/>
   <xacro:property name="meshes" value="file://$(find hexapod_description)/meshes"/>
@@ -20,5 +21,5 @@
   <!-- Base -->
   <xacro:base parent="base_footprint">
-    <origin xyz="0 0 0.4" rpy="0 0 0"/>
+    <origin xyz="0 0 ${HEXAPOD_HEIGHT}" rpy="0 0 0"/>
   </xacro:base>
   <!-- Arm -->

File: src/hexapod_description/robots/parts/sensors/sipeed_maixsense_a010.urdf.xacro (robot description, xacro)
@@ -61,5 +61,5 @@
     <always_on>true</always_on>
     <visualize>true</visualize>
-    <update_rate>10</update_rate> <!-- Max FPS according to spec -->
+    <update_rate>100</update_rate> <!-- Max FPS according to spec -->
     <topic>depth_camera/depth/image_raw</topic>
     <gz_frame_id>depth_camera_optical_frame</gz_frame_id>
