Commit message: Seperated robot into hexapod and arm

File: src/hexapod_description/robots/hexapod.urdf.xacro (robot description, xacro)
@@ -1,60 +1,50 @@
-<?xml version="1.0"?>
-<!-- Basic differential drive mobile base -->
-<robot xmlns:xacro="http://www.ros.org/wiki/xacro" name="hexapod">
-  <xacro:property name="description_package" value="$(find hexapod_description)"/>
-  <xacro:property name="HEXAPOD_HEIGHT" value="0.085"/>
-  <xacro:property name="robots" value="${description_package}/robots"/>
-  <xacro:property name="meshes" value="file://$(find hexapod_description)/meshes"/>
-  <xacro:include filename="$(find hexapod_description)/gazebo/hexapod.gazebo.xacro"/>
-  <xacro:include filename="$(find hexapod_description)/ros2_control/hexapod.ros2_control.xacro"/>
-  <xacro:include filename="$(find hexapod_description)/materials/hexapod.materials.xacro"/>
-  <xacro:include filename="${robots}/parts/base/base.urdf.xacro"/>
-  <xacro:include filename="${robots}/parts/arm/arm.urdf.xacro"/>
-  <xacro:include filename="${robots}/parts/leg/leg.urdf.xacro"/>
-  <xacro:include filename="${robots}/parts/sensors/sipeed_maixsense_a010.urdf.xacro"/>
+<?xml version="1.0" encoding="UTF-8"?>
+<!-- Basic differential drive mobile base --><robot name="hexapod" xmlns:xacro="http://www.ros.org/wiki/xacro">
+  <xacro:property name="description_package" value="$(find hexapod_description)"></xacro:property>
+  <xacro:property name="HEXAPOD_HEIGHT" value="0.085"></xacro:property>
+  <xacro:property name="robots" value="${description_package}/robots"></xacro:property>
+  <xacro:property name="meshes" value="file://$(find hexapod_description)/meshes"></xacro:property>
+  <xacro:include filename="$(find hexapod_description)/gazebo/hexapod.gazebo.xacro"></xacro:include>
+  <xacro:include filename="$(find hexapod_description)/ros2_control/hexapod.ros2_control.xacro"></xacro:include>
+  <xacro:include filename="$(find hexapod_description)/materials/hexapod.materials.xacro"></xacro:include>
+  <xacro:include filename="${robots}/parts/base/base.urdf.xacro"></xacro:include>
+  <xacro:include filename="${robots}/parts/leg/leg.urdf.xacro"></xacro:include>
+  <xacro:include filename="${robots}/parts/sensors/sipeed_maixsense_a010.urdf.xacro"></xacro:include>
   <!-- ================== ARGS ===================== -->
-  <xacro:arg name="initial_positions_file" default="initial_positions.yaml" />
+  <xacro:arg default="initial_positions.yaml" name="initial_positions_file"></xacro:arg>
   <!-- =============== Link & Joint =============== -->
   <!-- Base -->
-  <link name="base_footprint"/>
+  <link name="base_footprint"></link>
   <!--link name="base_footprint"/ -->
   <!-- Base -->
   <xacro:base parent="base_footprint">
-    <origin xyz="0 0 ${HEXAPOD_HEIGHT}" rpy="0 0 0"/>
+    <origin rpy="0 0 0" xyz="0 0 ${HEXAPOD_HEIGHT}"></origin>
   </xacro:base>
-  <!-- Arm -->
-  <xacro:arm parent="base_link">
-    <origin xyz="0.025588 -0.019423 0.0449" rpy="0 0 0"/>
-  </xacro:arm>
   <!-- Leg -->
   <xacro:leg parent="base_link" position="top" side="left">
-    <origin xyz="0.074451 0.046824 0.0297" rpy="0 0 ${-1/4*pi}"/>
+    <origin rpy="0 0 ${-1/4*pi}" xyz="0.074451 0.046824 0.0297"></origin>
   </xacro:leg>
   <!-- Leg -->
   <xacro:leg parent="base_link" position="mid" side="left">
-    <origin xyz="0.003612 0.056729 0.0306" rpy="0 0 ${0}"/>
+    <origin rpy="0 0 ${0}" xyz="0.003612 0.056729 0.0306"></origin>
   </xacro:leg>
   <!-- Leg -->
   <xacro:leg parent="base_link" position="bottom" side="left">
-    <origin xyz="-0.067095 0.047401 0.0297" rpy="0 0 ${1/4*pi}"/>
+    <origin rpy="0 0 ${1/4*pi}" xyz="-0.067095 0.047401 0.0297"></origin>
   </xacro:leg>
   <!-- Leg -->
   <xacro:leg parent="base_link" position="top" side="right">
-    <origin xyz="0.075633 -0.046741 0.0297" rpy="0 0 ${(1+1/4)*pi}"/>
+    <origin rpy="0 0 ${(1+1/4)*pi}" xyz="0.075633 -0.046741 0.0297"></origin>
   </xacro:leg>
   <!-- Leg -->
   <xacro:leg parent="base_link" position="mid" side="right">
-    <origin xyz="0.003574 -0.054899 0.0306" rpy="0 0 ${1*pi}"/>
+    <origin rpy="0 0 ${1*pi}" xyz="0.003574 -0.054899 0.0306"></origin>
   </xacro:leg>
   <!-- Leg -->
   <xacro:leg parent="base_link" position="bottom" side="right">
-    <origin xyz="-0.067095 -0.046741 0.0297" rpy="0 0 ${(1-1/4)*pi}"/>
+    <origin rpy="0 0 ${(1-1/4)*pi}" xyz="-0.067095 -0.046741 0.0297"></origin>
   </xacro:leg>
-  <!-- ================ Camera =============== -->
-  <xacro:camera parent="arm_retractor">
-    <origin xyz="-0.0125 0.0 0.055" rpy="0 ${-1/2*pi} ${-1/2*pi}"/>
-  </xacro:camera>
   <!-- =============== Gazebo =============== -->
-  <xacro:hexapod_gazebo/>
-  <xacro:hexapod_ros2_control name="FakeSystem" initial_positions_file="$(arg initial_positions_file)"/>
+  <xacro:hexapod_gazebo></xacro:hexapod_gazebo>
+  <xacro:hexapod_ros2_control initial_positions_file="$(arg initial_positions_file)" name="FakeSystem"></xacro:hexapod_ros2_control>
 </robot>

File: src/hexapod_description/robots/parts/arm/arm.urdf.xacro (robot description, xacro)
@@ -1,51 +1,44 @@
-<?xml version="1.0"?>
+<?xml version="1.0" encoding="UTF-8"?>
 <robot xmlns:xacro="http://ros.org/wiki/xacro">
   <xacro:macro name="arm" params="parent *joint_origin">
     <!-- Joints -->
     <joint name="arm_base_mount_joint" type="fixed">
-      <xacro:insert_block name="joint_origin"/>
-      <parent link="${parent}"/>
-      <child link="arm_base"/>
+      <xacro:insert_block name="joint_origin"></xacro:insert_block>
+      <parent link="${parent}"></parent>
+      <child link="arm_base"></child>
     </joint>
     <joint name="arm_rotator_joint" type="continuous">
-      <origin xyz="8.8e-05 0.019999 0.02995" rpy="0 0 0"/>
-      <parent link="arm_base"/>
-      <child link="arm_rotator"/>
-      <axis xyz="0.0 -0.0 -1.0"/>
-      <limit upper="1.570796" lower="-1.570796" effort="100" velocity="100"/>
+      <origin rpy="0 0 0" xyz="8.8e-05 0.019999 0.02995"></origin>
+      <parent link="arm_base"></parent>
+      <child link="arm_rotator"></child>
+      <axis xyz="0.0 -0.0 -1.0"></axis>
+      <limit effort="100" lower="-1.570796" upper="1.570796" velocity="100"></limit>
     </joint>
     <joint name="arm_abductor_joint" type="revolute">
-      <origin xyz="0.014582 0.00069 0.013923" rpy="0 0 0"/>
-      <parent link="arm_rotator"/>
-      <child link="arm_abductor"/>
-      <axis xyz="-1.0 0.0 -0.0"/>
-      <limit upper="1.570796" lower="-1.570796" effort="100" velocity="100"/>
+      <origin rpy="0 0 0" xyz="0.014582 0.00069 0.013923"></origin>
+      <parent link="arm_rotator"></parent>
+      <child link="arm_abductor"></child>
+      <axis xyz="-1.0 0.0 -0.0"></axis>
+      <limit effort="100" lower="-1.570796" upper="1.570796" velocity="100"></limit>
     </joint>
-    <joint name="arm_retractor_joint" type="revolute">
-      <origin xyz="-0.000401 0.0 0.046709" rpy="0 0 0"/>
-      <parent link="arm_abductor"/>
-      <child link="arm_retractor"/>
-      <axis xyz="-0.999993 0.0 -0.003676"/>
-      p
-      <limit upper="1.570796" lower="-1.570796" effort="100" velocity="100"/>
-    </joint>
+    <joint name="arm_retractor_joint" type="revolute"><origin rpy="0 0 0" xyz="-0.000401 0.0 0.046709"></origin> <parent link="arm_abductor"></parent> <child link="arm_retractor"></child> <axis xyz="-0.999993 0.0 -0.003676"></axis> p <limit effort="100" lower="-1.570796" upper="1.570796" velocity="100"></limit></joint>
     <!-- Links -->
     <link name="arm_rotator">
       <inertial>
-        <origin xyz="-0.00046642883527773724 0.0027188082250819237 0.00576546998065737" rpy="0 0 0"/>
-        <mass value="0.02623546025799875"/>
-        <inertia ixx="4e-06" iyy="4e-06" izz="5e-06" ixy="0.0" iyz="-0.0" ixz="0.0"/>
+        <origin rpy="0 0 0" xyz="-0.00046642883527773724 0.0027188082250819237 0.00576546998065737"></origin>
+        <mass value="0.02623546025799875"></mass>
+        <inertia ixx="4e-06" ixy="0.0" ixz="0.0" iyy="4e-06" iyz="-0.0" izz="5e-06"></inertia>
       </inertial>
       <visual>
-        <origin xyz="-0.025676 -0.000576 -0.07485" rpy="0 0 0"/>
+        <origin rpy="0 0 0" xyz="-0.025676 -0.000576 -0.07485"></origin>
         <geometry>
-          <mesh filename="${meshes}/visual/rotator.stl" scale="0.001 0.001 0.001"/>
+          <mesh filename="${meshes}/visual/rotator.stl" scale="0.001 0.001 0.001"></mesh>
         </geometry>
-        <material name="PLA"/>
+        <material name="PLA"></material>
       </visual>
       <collision>
-        <origin xyz="-0.025676 -0.000576 -0.07485" rpy="0 0 0"/>
+        <origin rpy="0 0 0" xyz="-0.025676 -0.000576 -0.07485"></origin>
         <geometry>
-          <mesh filename="${meshes}/collision/rotator.stl" scale="0.001 0.001 0.001"/>
+          <mesh filename="${meshes}/collision/rotator.stl" scale="0.001 0.001 0.001"></mesh>
         </geometry>
       </collision>
@@ -53,19 +46,19 @@
     <link name="arm_abductor">
       <inertial>
-        <origin xyz="-0.014167725035919117 3.5639852713031765e-07 0.031090662760010462" rpy="0 0 0"/>
-        <mass value="0.016534189067873267"/>
-        <inertia ixx="5e-06" iyy="7e-06" izz="2e-06" ixy="-0.0" iyz="-0.0" ixz="1e-06"/>
+        <origin rpy="0 0 0" xyz="-0.014167725035919117 3.5639852713031765e-07 0.031090662760010462"></origin>
+        <mass value="0.016534189067873267"></mass>
+        <inertia ixx="5e-06" ixy="-0.0" ixz="1e-06" iyy="7e-06" iyz="-0.0" izz="2e-06"></inertia>
       </inertial>
       <visual>
-        <origin xyz="-0.040258 -0.001266 -0.088773" rpy="0 0 0"/>
+        <origin rpy="0 0 0" xyz="-0.040258 -0.001266 -0.088773"></origin>
         <geometry>
-          <mesh filename="${meshes}/visual/abductor.stl" scale="0.001 0.001 0.001"/>
+          <mesh filename="${meshes}/visual/abductor.stl" scale="0.001 0.001 0.001"></mesh>
         </geometry>
-        <material name="PLA"/>
+        <material name="PLA"></material>
       </visual>
       <collision>
-        <origin xyz="-0.040258 -0.001266 -0.088773" rpy="0 0 0"/>
+        <origin rpy="0 0 0" xyz="-0.040258 -0.001266 -0.088773"></origin>
         <geometry>
-          <mesh filename="${meshes}/collision/abductor.stl" scale="0.001 0.001 0.001"/>
+          <mesh filename="${meshes}/collision/abductor.stl" scale="0.001 0.001 0.001"></mesh>
         </geometry>
       </collision>
@@ -73,19 +66,19 @@
     <link name="arm_retractor">
       <inertial>
-        <origin xyz="-0.011027322351092845 -5.220911472792085e-05 0.023364114206742087" rpy="0 0 0"/>
-        <mass value="0.015328010788351278"/>
-        <inertia ixx="3e-06" iyy="5e-06" izz="4e-06" ixy="0.0" iyz="0.0" ixz="-0.0"/>
+        <origin rpy="0 0 0" xyz="-0.011027322351092845 -5.220911472792085e-05 0.023364114206742087"></origin>
+        <mass value="0.015328010788351278"></mass>
+        <inertia ixx="3e-06" ixy="0.0" ixz="-0.0" iyy="5e-06" iyz="0.0" izz="4e-06"></inertia>
       </inertial>
       <visual>
-        <origin xyz="-0.039857 -0.001266 -0.135482" rpy="0 0 0"/>
+        <origin rpy="0 0 0" xyz="-0.039857 -0.001266 -0.135482"></origin>
         <geometry>
-          <mesh filename="${meshes}/visual/retractor.stl" scale="0.001 0.001 0.001"/>
+          <mesh filename="${meshes}/visual/retractor.stl" scale="0.001 0.001 0.001"></mesh>
         </geometry>
-        <material name="PLA"/>
+        <material name="PLA"></material>
       </visual>
       <collision>
-        <origin xyz="-0.039857 -0.001266 -0.135482" rpy="0 0 0"/>
+        <origin rpy="0 0 0" xyz="-0.039857 -0.001266 -0.135482"></origin>
         <geometry>
-          <mesh filename="${meshes}/collision/retractor.stl" scale="0.001 0.001 0.001"/>
+          <mesh filename="${meshes}/collision/retractor.stl" scale="0.001 0.001 0.001"></mesh>
         </geometry>
       </collision>
@@ -93,19 +86,19 @@
     <link name="arm_base">
       <inertial>
-        <origin xyz="0.004115093716825637 0.020000308654227843 0.01035421864114821" rpy="0 0 0"/>
-        <mass value="0.014628769254330782"/>
-        <inertia ixx="2e-06" iyy="3e-06" izz="2e-06" ixy="0.0" iyz="0.0" ixz="-0.0"/>
+        <origin rpy="0 0 0" xyz="0.004115093716825637 0.020000308654227843 0.01035421864114821"></origin>
+        <mass value="0.014628769254330782"></mass>
+        <inertia ixx="2e-06" ixy="0.0" ixz="-0.0" iyy="3e-06" iyz="0.0" izz="2e-06"></inertia>
       </inertial>
       <visual>
-        <origin xyz="-0.025588 0.019423 -0.0449" rpy="0 0 0"/>
+        <origin rpy="0 0 0" xyz="-0.025588 0.019423 -0.0449"></origin>
         <geometry>
-          <mesh filename="${meshes}/visual/base.stl" scale="0.001 0.001 0.001"/>
+          <mesh filename="${meshes}/visual/base.stl" scale="0.001 0.001 0.001"></mesh>
         </geometry>
-        <material name="PLA"/>
+        <material name="PLA"></material>
       </visual>
       <collision>
-        <origin xyz="-0.025588 0.019423 -0.0449" rpy="0 0 0"/>
+        <origin rpy="0 0 0" xyz="-0.025588 0.019423 -0.0449"></origin>
         <geometry>
-          <mesh filename="${meshes}/collision/base.stl" scale="0.001 0.001 0.001"/>
+          <mesh filename="${meshes}/collision/base.stl" scale="0.001 0.001 0.001"></mesh>
         </geometry>
       </collision>

File: src/hexapod_description/ros2_control/hexapod.ros2_control.xacro (robot description, xacro)
@@ -6,4 +6,5 @@
         <param name="min">-1.5</param>
         <param name="max">1.5</param>
+        <!--       <param name="initial_value">${initial_positions['top_left_rotate_joint']}</param> -->
       </command_interface>
       <state_interface name="position"></state_interface>
@@ -15,12 +16,4 @@
     </plugin>
   </gazebo>
-  <!-- Code to set params from .yaml file -->
-  <!-- <joint name="top_left_rotate_joint"> -->
-  <!--     <command_interface name="position"/> -->
-  <!--     <state_interface name="position"> -->
-  <!--       <param name="initial_value">${initial_positions['top_left_rotate_joint']}</param> -->
-  <!--     </state_interface> -->
-  <!--     <state_interface name="velocity"/> -->
-  <!-- </joint> -->
   <xacro:macro name="hexapod_ros2_control" params="name initial_positions_file">
     <xacro:property name="initial_positions" value="${xacro.load_yaml(initial_positions_file)['initial_positions']}"></xacro:property>
@@ -29,7 +22,4 @@
         <plugin>gz_ros2_control/GazeboSimSystem</plugin>
       </hardware>
-      <xacro:joint name="arm_rotator_joint"></xacro:joint>
-      <xacro:joint name="arm_abductor_joint"></xacro:joint>
-      <xacro:joint name="arm_retractor_joint"></xacro:joint>
       <xacro:joint name="top_left_rotate_joint"></xacro:joint>
       <xacro:joint name="top_left_abduct_joint"></xacro:joint>
